File: Orbit-PCB/Orbit.sch (KiCad schematic (older format))
At the start: 130 parts

Commit message: Assign footprints
Parts:
- C1, C2, C3, C4, C5, C6, C7: renamed from C?; footprint (none) -> Capacitors_SMD:C_0805
- D1, D10, D11, D12, D13, D14, D15, D16, D17, D18, D19, D2, D20, D21, D22, D23, D24, D25, D26, D27, D28, D29, D3, D30, D31, D32, D33, D34, D35, D4, D5, D6, D7, D8, D9: renamed from D?; footprint (none) -> Diodes_SMD:D_SOD-123
- F1: renamed from F?; footprint (none) -> Fuse_Holders_and_Fuses:Fuse_SMD1206_Reflow
- J1: renamed from J?; footprint (none) -> locallib:PJ-3200B-4A
- MX1, MX10, MX11, MX12, MX13, MX14, MX15, MX16, MX17, MX18, MX19, MX2, MX20, MX21, MX22, MX23, MX24, MX25, MX26, MX27, MX28, MX29, MX3, MX30, MX31, MX32, MX33, MX34, MX35, MX4, MX5, MX6, MX7, MX8, MX9: renamed from MX?; footprint (none) -> MX_Alps_Hybrid:MX-1U
- R1, R10, R11, R12, R13, R14, R15, R16, R17, R18, R19, R2, R20, R21, R22, R23, R24, R25, R26, R27, R28, R29, R3, R30, R31, R32, R33, R34, R35, R36, R37, R38, R39, R4, R40, R41, R42, R43, R44, R5, R6, R7, R8, R9: renamed from R?; footprint (none) -> Resistors_SMD:R_0805
- SW1: renamed from SW?; footprint (none) -> Molex-0548190589:PushButton_6x6mm_TH_Pretty
- U2: renamed from U?; footprint (none) -> locallib:SOT143B
- USB1: renamed from USB?; footprint (none) -> Type-C:HRO-TYPE-C-31-M-12-Assembly
- Y1: renamed from Y?; footprint (none) -> Crystals:Crystal_SMD_3225-4pin_3.2x2.5mm
- gave numbers to parts that had none: 3

Commit message: Route one half
Parts:
- removed D29: SOD-123, Diodes_SMD:D_SOD-123, symbol Device:D_Small
- removed MX29: MX-1U, MX_Alps_Hybrid:MX-1U, symbol MX_Alps_Hybrids:MX-1U
- added D35: LED_1.8mm, LEDs:LED_D3.0mm, symbol Device:LED_Small
- C1, C2, C3, C4, C5, C6, C7: footprint Capacitors_SMD:C_0805 -> Capacitors_SMD:C_0603
- J2: footprint (none) -> Molex-0548190589:Reset_Pretty-Mask
- MX34: renamed from MX35; value MX-1U -> MX-1.5U; footprint MX_Alps_Hybrid:MX-1U -> MX_Alps_Hybrid:MX-1.5U-Vertical
- Q1: footprint Package_TO_SOT_SMD:SOT-23 -> TO_SOT_Packages_SMD:SOT-23
- R33: value 470 -> 1k
- SW1: footprint Molex-0548190589:PushButton_6x6mm_TH_Pretty -> Molex-0548190589:SKQG-1155865
- U1: value ATmega32U4-AU -> ATmega32U4-MU; footprint Housings_QFP:TQFP-44_10x10mm_Pitch0.8mm -> Housings_DFN_QFN:QFN-44-1EP_7x7mm_Pitch0.5mm
- renumbered D30 to D29, D31 to D30, D32 to D31, D33 to D32, D34 to D33, D35 to D34, MX30 to MX29, MX31 to MX30, MX32 to MX31, MX33 to MX32, MX34 to MX33
Connections:
- net labels added: LEDIND
- wire segments 303 -> 300
Other:
- note added: "0.1"
- note added: "1 1"
- note added: "2018-09-02"
- note added: "Credits to \ncrkbd by foostan - Design inspiration and base\nIris by Bakingpy - Schematic reference"
- note added: "Indicator LED"
- note added: "Orbit - LEFT HALF by ai03"

Commit message: Round corner and route indicator LED
Changed lines of the file:
@@
 Text GLabel 4100 3850 2    50   Input ~ 0
 ROW4
+Text GLabel 4100 2950 2    50   Input ~ 0
+LEDIND
 $EndSCHEMATC

Commit message: Both halves roughly complete, begin cleaning
Parts:
- added C10: 1uF, Capacitors_SMD:C_0603, symbol Device:C_Small
- added C11, C12, C13: 0.1uF, Capacitors_SMD:C_0603, symbol Device:C_Small
- added C14: 10uF, Capacitors_SMD:C_0603, symbol Device:C_Small
- added C8, C9: 22pF, Capacitors_SMD:C_0603, symbol Device:C_Small
- added D36, D37, D38, D39, D40, D41, D42, D43, D44, D45, D46, D47, D48, D49, D50, D51, D52, D53, D54, D55, D56, D57, D58, D59, D60, D61, D62, D63, D64, D65, D66, D67, D68, D69: SOD-123, Diodes_SMD:D_SOD-123, symbol Device:D_Small
- added D70: LED_1.8mm, LEDs:LED_D3.0mm, symbol Device:LED_Small
- added F2: 500mA, Fuse_Holders_and_Fuses:Fuse_SMD1206_Reflow, symbol Device:Polyfuse_Small
- added J10, J13, J14, J15, J16, J17, J18, J19, J20, J3, J4, J5, J6, J7, J8, J9: Breakaway_Tabs, locallib:breakaway-mousebites, symbol Connector_Generic:Conn_01x01
- added J11: PJ-3200B-4A, locallib:PJ-3200B-4A, symbol Connector_Generic:Conn_01x04
- added J12: AVR-ISP-6, Molex-0548190589:Reset_Pretty-Mask, symbol Connector:AVR-ISP-6
- added MX35, MX36, MX37, MX38, MX39, MX40, MX41, MX42, MX43, MX44, MX45, MX46, MX47, MX48, MX49, MX50, MX51, MX52, MX53, MX54, MX55, MX56, MX57, MX58, MX59, MX60, MX61, MX62, MX64, MX65, MX66, MX67, MX68: MX-1U, MX_Alps_Hybrid:MX-1U, symbol MX_Alps_Hybrids:MX-1U
- added MX63: MX-1.5U, MX_Alps_Hybrid:MX-1.5U-Vertical, symbol MX_Alps_Hybrids:MX-1U
- added Q2: 2N7002, TO_SOT_Packages_SMD:SOT-23, symbol Transistor_FET:2N7002
- added R45, R67: 10k, Resistors_SMD:R_0805, symbol Device:R_Small
- added R46, R47, R48, R49, R50, R51, R52, R53, R54, R55, R56, R57, R58, R59, R60, R61, R62, R63, R64, R65, R66, R68, R69, R70, R71, R72, R73, R74, R75, R76, R77, R78, R79, R80: 470, Resistors_SMD:R_0805, symbol Device:R_Small
- added R81, R82: 1k, Resistors_SMD:R_0805, symbol Device:R_Small
- added R83, R84: 22, Resistors_SMD:R_0805, symbol Device:R_Small
- added R85, R86: 5.1k, Resistors_SMD:R_0805, symbol Device:R_Small
- added SW2: SW_Push, Molex-0548190589:SKQG-1155865, symbol Switch:SW_Push
- added U3: ATmega32U4-MU, Housings_DFN_QFN:QFN-44-1EP_7x7mm_Pitch0.5mm, symbol MCU_Microchip_ATmega:ATmega32U4-AU
- added U4: PRTR5V0U2X, locallib:SOT143B, symbol ai03-locallib:PRTR5V0U2X
- added USB2: HRO-TYPE-C-31-M-12, Type-C:HRO-TYPE-C-31-M-12-Assembly, symbol Type-C:HRO-TYPE-C-31-M-12
- added Y2: 16MHz, Crystals:Crystal_SMD_2520-4pin_2.5x2.0mm, symbol Device:Crystal_GND24_Small
- Y1: footprint Crystals:Crystal_SMD_3225-4pin_3.2x2.5mm -> Crystals:Crystal_SMD_2520-4pin_2.5x2.0mm
Connections:
- net labels added: +5VA, COL0-R, COL1-R, COL2-R, COL3-R, COL4-R, COL5-R, COL6-R, D+-R, D--R, GNDA, LEDGND-R, LEDIND-R, LEDPWM-R, MISO-R, MOSI-R, RESET-R, ROW0-R, ROW1-R, ROW2-R, ROW3-R, ROW4-R, SCK-R, SCL-R, SDA-R, VDD
- wire segments 300 -> 595
- no-connect marks 3 -> 22
Other:
- note added: "Credits to \ncrkbd by foostan - Design inspiration and fork base\nIris by Bakingpy - Schematic reference"
- note added: "Extra Hardware"
- note added: "LEFT HAND SCHEMATIC"
- note added: "Orbit by ai03"
- note added: "RIGHT HAND SCHEMATIC\n\nPower net changes:\nVCC -> VDD\nGND -> GNDA\n+5V -> +5VA\nto prevent kicad from complaining about no connections between halves"
- note removed: "Credits to \ncrkbd by foostan - Design inspiration and base\nIris by Bakingpy - Schematic reference"
- note removed: "Orbit - LEFT HALF by ai03"

Commit message: Add left/right hand detection pullup/downs
Parts:
- added J21: Conn_01x01, Mounting_Holes:MountingHole_3.5mm_Pad_Via, symbol Connector_Generic:Conn_01x01
- added MH1, MH2: HOLE, Mounting_Holes:MountingHole_5mm, symbol Connector_Generic:Conn_01x01
- added R87, R88: 10k, Resistors_SMD:R_0805, symbol Device:R_Small
Connections:
- net labels added: GNDS, HDETECT, HDETECT-R
- wire segments 595 -> 599
- no-connect marks 22 -> 24
Other:
- note added: "Extras"
- note added: "Half Detection"
- note added: "Passthrough Holes"
- note added: "Passthrough Holes\n"
- note added: "Read low = Right hand"
Changed lines of the file:
@@
 Wire Wire Line
 	3225 7300 3275 7300
-Wire Notes Line
-	7750 6400 5650 6400
 $Comp
 L Device:R_Small R33
@@
 Wire Wire Line
 	3225 14875 3275 14875
-Wire Notes Line
-	7750 13975 5650 13975
 $Comp
 L Device:R_Small R82
@@
 	9150 11950 9750 11950
 Connection ~ 9750 11950
+Wire Notes Line
+	14300 675  16150 675
+Wire Notes Line
+	16150 675  16150 2325
+Wire Notes Line
+	16150 2325 14300 2325
+Wire Notes Line
+	14300 2325 14300 675
+$Comp
+L Connector_Generic:Conn_01x01 J21
+U 1 1 5C31FC53
+P 14875 1050
+F 0 "J21" H 14955 1092 50  0000 L CNN
+F 1 "Conn_01x01" H 14955 1001 50  0000 L CNN
+F 2 "Mounting_Holes:MountingHole_3.5mm_Pad_Via" H 14875 1050 50  0001 C CNN
+F 3 "~" H 14875 1050 50  0001 C CNN
+	1    14875 1050
+	1    0    0    -1
+$EndComp
+Text Notes 14325 775  0    50   ~ 0
+Extras
+$Comp
+L power:GNDS #PWR01
+U 1 1 5C3200EF
+P 14675 1050
+F 0 "#PWR01" H 14675 800 50  0001 C CNN
+F 1 "GNDS" H 14680 877 50  0000 C CNN
+F 2 "" H 14675 1050 50  0001 C CNN
+F 3 "" H 14675 1050 50  0001 C CNN
+	1    14675 1050
+	1    0    0    -1
+$EndComp
+Wire Notes Line
+	9175 5250 9175 7700
+Wire Notes Line
+	5650 6400 9175 6400
+Wire Notes Line
+	9175 12825 9175 15275
+Wire Notes Line
+	5650 13975 9175 13975
+Text Notes 7775 12925 0    50   ~ 0
+Passthrough Holes\n
+Text Notes 7775 5350 0    50   ~ 0
+Passthrough Holes
+$Comp
+L Connector_Generic:Conn_01x01 MH1
+U 1 1 5C5F2D6B
+P 8150 5600
+F 0 "MH1" H 8229 5642 50  0000 L CNN
+F 1 "HOLE" H 8229 5551 50  0000 L CNN
+F 2 "Mounting_Holes:MountingHole_5mm" H 8150 5600 50  0001 C CNN
+F 3 "~" H 8150 5600 50  0001 C CNN
+	1    8150 5600
+	1    0    0    -1
+$EndComp
+NoConn ~ 7950 5600
+$Comp
+L Connector_Generic:Conn_01x01 MH2
+U 1 1 5C7F1ECF
+P 8175 13150
+F 0 "MH2" H 8254 13192 50  0000 L CNN
+F 1 "HOLE" H 8254 13101 50  0000 L CNN
+F 2 "Mounting_Holes:MountingHole_5mm" H 8175 13150 50  0001 C CNN
+F 3 "~" H 8175 13150 50  0001 C CNN
+	1    8175 13150
+	1    0    0    -1
+$EndComp
+NoConn ~ 7975 13150
+Text Notes 7775 6500 0    50   ~ 0
+Half Detection
+Text GLabel 8250 6875 0    50   Input ~ 0
+HDETECT
+$Comp
+L Device:R_Small R87
+U 1 1 5C98FB97
+P 8450 6875
+F 0 "R87" V 8254 6875 50  0000 C CNN
+F 1 "10k" V 8345 6875 50  0000 C CNN
+F 2 "Resistors_SMD:R_0805" H 8450 6875 50  0001 C CNN
+F 3 "~" H 8450 6875 50  0001 C CNN
+	1    8450 6875
+	0    1    1    0
+$EndComp
+Wire Wire Line
+	8350 6875 8250 6875
+Wire Wire Line
+	8675 6875 8550 6875
+$Comp
+L power:+5V #PWR0145
+U 1 1 5CA5E548
+P 8675 6875
+F 0 "#PWR0145" H 8675 6725 50  0001 C CNN
+F 1 "+5V" H 8690 7048 50  0000 C CNN
+F 2 "" H 8675 6875 50  0001 C CNN
+F 3 "" H 8675 6875 50  0001 C CNN
+	1    8675 6875
+	1    0    0    -1
+$EndComp
+Text Notes 7775 7175 0    50   ~ 0
+Read low = Right hand
+Text Notes 7775 14075 0    50   ~ 0
+Half Detection
+Text GLabel 8250 14450 0    50   Input ~ 0
+HDETECT-R
+$Comp
+L Device:R_Small R88
+U 1 1 5CA60302
+P 8450 14450
+F 0 "R88" V 8254 14450 50  0000 C CNN
+F 1 "10k" V 8345 14450 50  0000 C CNN
+F 2 "Resistors_SMD:R_0805" H 8450 14450 50  0001 C CNN
+F 3 "~" H 8450 14450 50  0001 C CNN
+	1    8450 14450
+	0    1    1    0
+$EndComp
+Wire Wire Line
+	8350 14450 8250 14450
+Wire Wire Line
+	8675 14450 8550 14450
+Text Notes 7775 14750 0    50   ~ 0
+Read low = Right hand
+$Comp
+L power:GNDA #PWR0146
+U 1 1 5CAC829D
+P 8675 14450
+F 0 "#PWR0146" H 8675 14200 50  0001 C CNN
+F 1 "GNDA" H 8680 14277 50  0000 C CNN
+F 2 "" H 8675 14450 50  0001 C CNN
+F 3 "" H 8675 14450 50  0001 C CNN
+	1    8675 14450
+	1    0    0    -1
+$EndComp
+Text GLabel 4100 3050 2    50   Input ~ 0
+HDETECT
+Text GLabel 4100 10625 2    50   Input ~ 0
+HDETECT-R
 $EndSCHEMATC

Commit message: Add 2U compat
Parts:
- removed J16, J4, J8: Breakaway_Tabs, locallib:breakaway-mousebites, symbol Connector_Generic:Conn_01x01
- added MXE-1, MXE-2: MX-2U, MX_Alps_Hybrid:MX-2U, symbol MX_Alps_Hybrids:MX-1U
- added MXE-3, MXE-4, MXE-5, MXE-6: MX-2U, MX_Alps_Hybrid:MX-2U-ReversedStabilizers, symbol MX_Alps_Hybrids:MX-1U
Connections:
- wire segments 599 -> 623
- no-connect marks 24 -> 21
Other:
- moved on the sheet: J15
Changed lines of the file:
@@
 	9175 4925 9775 4925
 Wire Wire Line
-	9775 4925 9775 4075
+	9775 4925 9775 4725
 Connection ~ 9175 2125
 Wire Wire Line
@@
 NoConn ~ 5800 6650
 $Comp
-L Connector_Generic:Conn_01x01 J4
-U 1 1 5BBF4619
-P 6000 6825
-F 0 "J4" H 6079 6867 50  0000 L CNN
-F 1 "Breakaway_Tabs" H 6079 6776 50  0000 L CNN
-F 2 "locallib:breakaway-mousebites" H 6000 6825 50  0001 C CNN
-F 3 "~" H 6000 6825 50  0001 C CNN
-	1    6000 6825
-	1    0    0    -1
-$EndComp
-$Comp
 L Connector_Generic:Conn_01x01 J5
 U 1 1 5BBF47C0
@@
 NoConn ~ 5800 7175
 NoConn ~ 5800 7000
-NoConn ~ 5800 6825
 $Comp
 L Connector_Generic:Conn_01x01 J7
@@
 NoConn ~ 6775 6650
 $Comp
-L Connector_Generic:Conn_01x01 J8
-U 1 1 5BC3C168
-P 6975 6825
-F 0 "J8" H 7054 6867 50  0000 L CNN
-F 1 "Breakaway_Tabs" H 7054 6776 50  0000 L CNN
-F 2 "locallib:breakaway-mousebites" H 6975 6825 50  0001 C CNN
-F 3 "~" H 6975 6825 50  0001 C CNN
-	1    6975 6825
-	1    0    0    -1
-$EndComp
-$Comp
 L Connector_Generic:Conn_01x01 J9
 U 1 1 5BC3C16F
@@
 NoConn ~ 6775 7175
 NoConn ~ 6775 7000
-NoConn ~ 6775 6825
 $Comp
 L MCU_Microchip_ATmega:ATmega32U4-AU U3
@@
 L Connector_Generic:Conn_01x01 J15
 U 1 1 5BCD1D42
-P 6000 14400
-F 0 "J15" H 6079 14442 50  0000 L CNN
-F 1 "Breakaway_Tabs" H 6079 14351 50  0000 L CNN
-F 2 "locallib:breakaway-mousebites" H 6000 14400 50  0001 C CNN
-F 3 "~" H 6000 14400 50  0001 C CNN
-	1    6000 14400
+P 14650 2150
+F 0 "J15" H 14729 2192 50  0000 L CNN
+F 1 "Breakaway_Tabs" H 14729 2101 50  0000 L CNN
+F 2 "locallib:breakaway-mousebites" H 14650 2150 50  0001 C CNN
+F 3 "~" H 14650 2150 50  0001 C CNN
+	1    14650 2150
 	1    0    0    -1
 $EndComp
@@
 NoConn ~ 5800 14750
 NoConn ~ 5800 14575
-NoConn ~ 5800 14400
+NoConn ~ 14450 2150
 $Comp
 L Connector_Generic:Conn_01x01 J14
@@
 NoConn ~ 6775 14225
 $Comp
-L Connector_Generic:Conn_01x01 J16
-U 1 1 5BCD1D62
-P 6975 14400
-F 0 "J16" H 7054 14442 50  0000 L CNN
-F 1 "Breakaway_Tabs" H 7054 14351 50  0000 L CNN
-F 2 "locallib:breakaway-mousebites" H 6975 14400 50  0001 C CNN
-F 3 "~" H 6975 14400 50  0001 C CNN
-	1    6975 14400
-	1    0    0    -1
-$EndComp
-$Comp
 L Connector_Generic:Conn_01x01 J18
 U 1 1 5BCD1D69
@@
 NoConn ~ 6775 14750
 NoConn ~ 6775 14575
-NoConn ~ 6775 14400
 Text Notes 13050 7650 0    50   ~ 10
 LEFT HAND SCHEMATIC
@@
 Connection ~ 12175 11650
 Wire Wire Line
-	12175 11650 12175 12500
+	12175 11650 12175 12275
 Wire Wire Line
 	12150 11950 13325 11950
@@
 Text GLabel 4100 10625 2    50   Input ~ 0
 HDETECT-R
+$Comp
+L MX_Alps_Hybrids:MX-1U MXE-1
+U 1 1 5CC78A6A
+P 8575 2100
+F 0 "MXE-1" H 8661 2317 60  0000 C CNN
+F 1 "MX-2U" H 8661 2243 20  0000 C CNN
+F 2 "MX_Alps_Hybrid:MX-2U" H 8550 2075 60  0001 C CNN
+F 3 "" H 8550 2075 60  0001 C CNN
+	1    8575 2100
+	1    0    0    -1
+$EndComp
+$Comp
+L MX_Alps_Hybrids:MX-1U MXE-2
+U 1 1 5CC79D1C
+P 8575 3400
+F 0 "MXE-2" H 8661 3617 60  0000 C CNN
+F 1 "MX-2U" H 8661 3543 20  0000 C CNN
+F 2 "MX_Alps_Hybrid:MX-2U" H 8550 3375 60  0001 C CNN
+F 3 "" H 8550 3375 60  0001 C CNN
+	1    8575 3400
+	1    0    0    -1
+$EndComp
+$Comp
+L MX_Alps_Hybrids:MX-1U MXE-3
+U 1 1 5CC7A722
+P 9650 4700
+F 0 "MXE-3" H 9736 4917 60  0000 C CNN
+F 1 "MX-2U" H 9736 4843 20  0000 C CNN
+F 2 "MX_Alps_Hybrid:MX-2U-ReversedStabilizers" H 9625 4675 60  0001 C CNN
+F 3 "" H 9625 4675 60  0001 C CNN
+	1    9650 4700
+	1    0    0    -1
+$EndComp
+Connection ~ 9775 4725
+Wire Wire Line
+	9775 4725 9775 4075
+$Comp
+L MX_Alps_Hybrids:MX-1U MXE-6
+U 1 1 5CC7BD3E
+P 12050 12250
+F 0 "MXE-6" H 12136 12467 60  0000 C CNN
+F 1 "MX-2U" H 12136 12393 20  0000 C CNN
+F 2 "MX_Alps_Hybrid:MX-2U-ReversedStabilizers" H 12025 12225 60  0001 C CNN
+F 3 "" H 12025 12225 60  0001 C CNN
+	1    12050 12250
+	1    0    0    -1
+$EndComp
+Connection ~ 12175 12275
+Wire Wire Line
+	12175 12275 12175 12500
+$Comp
+L MX_Alps_Hybrids:MX-1U MXE-4
+U 1 1 5CC7DA98
+P 13100 9675
+F 0 "MXE-4" H 13186 9892 60  0000 C CNN
+F 1 "MX-2U" H 13186 9818 20  0000 C CNN
+F 2 "MX_Alps_Hybrid:MX-2U-ReversedStabilizers" H 13075 9650 60  0001 C CNN
+F 3 "" H 13075 9650 60  0001 C CNN
+	1    13100 9675
+	1    0    0    -1
+$EndComp
+$Comp
+L MX_Alps_Hybrids:MX-1U MXE-5
+U 1 1 5CC7F491
+P 13100 10975
+F 0 "MXE-5" H 13186 11192 60  0000 C CNN
+F 1 "MX-2U" H 13186 11118 20  0000 C CNN
+F 2 "MX_Alps_Hybrid:MX-2U-ReversedStabilizers" H 13075 10950 60  0001 C CNN
+F 3 "" H 13075 10950 60  0001 C CNN
+	1    13100 10975
+	1    0    0    -1
+$EndComp
+Wire Wire Line
+	9225 3375 8750 3375
+Connection ~ 9225 3375
+Wire Wire Line
+	9175 3425 8700 3425
+Wire Wire Line
+	8950 3575 8550 3575
+Connection ~ 8950 3575
+Wire Wire Line
+	8600 3525 9075 3525
+Connection ~ 9075 3525
+Wire Wire Line
+	9225 2075 8750 2075
+Wire Wire Line
+	8700 2125 9175 2125
+Wire Wire Line
+	9075 2225 8600 2225
+Connection ~ 9075 2225
+Wire Wire Line
+	8550 2275 8950 2275
+Connection ~ 8950 2275
+Wire Wire Line
+	9825 4025 9825 4675
+Connection ~ 9825 4025
+Wire Wire Line
+	9675 4825 9675 4175
+Connection ~ 9675 4175
+Wire Wire Line
+	9625 4225 9625 4875
+Connection ~ 9625 4225
+Wire Wire Line
+	12825 9650 13275 9650
+Wire Wire Line
+	13225 9700 12775 9700
+Wire Wire Line
+	12750 9800 13125 9800
+Connection ~ 12750 9800
+Wire Wire Line
+	13075 9850 12625 9850
+Connection ~ 12625 9850
+Wire Wire Line
+	13275 10950 12825 10950
+Connection ~ 12825 10950
+Wire Wire Line
+	12775 11000 13225 11000
+Wire Wire Line
+	13125 11100 12750 11100
+Connection ~ 12750 11100
+Wire Wire Line
+	12625 11150 13075 11150
+Connection ~ 12625 11150
+Wire Wire Line
+	12225 11600 12225 12225
+Connection ~ 12225 11600
+Wire Wire Line
+	12075 12375 12075 11750
+Connection ~ 12075 11750
+Wire Wire Line
+	12025 11800 12025 12425
+Connection ~ 12025 11800
 $EndSCHEMATC

Commit message: Fix 1.5U spacebar alps support
Parts:
- removed J15: Breakaway_Tabs, locallib:breakaway-mousebites, symbol Connector_Generic:Conn_01x01
- removed J21: Conn_01x01, Mounting_Holes:MountingHole_3.5mm_Pad_Via, symbol Connector_Generic:Conn_01x01
- added MXA1, MXA2: ALPS-1.5U, MX_Alps_Hybrid:ALPS-1.5U, symbol MX_Alps_Hybrids:MX-1U
- MX34, MX63: footprint MX_Alps_Hybrid:MX-1.5U-Vertical -> MX_Alps_Hybrid:MXOnly-1.5U-Vertical
Connections:
- net labels removed: GNDS
- wire segments 623 -> 635
- no-connect marks 21 -> 20
Other:
- note removed: "Extras"
Changed lines of the file:
@@
 F 0 "MX34" H 12736 4267 60  0000 C CNN
 F 1 "MX-1.5U" H 12736 4193 20  0000 C CNN
-F 2 "MX_Alps_Hybrid:MX-1.5U-Vertical" H 12625 4025 60  0001 C CNN
+F 2 "MX_Alps_Hybrid:MXOnly-1.5U-Vertical" H 12625 4025 60  0001 C CNN
 F 3 "" H 12625 4025 60  0001 C CNN
 	1    12650 4050
@@
 F 0 "MX63" H 9136 11842 60  0000 C CNN
 F 1 "MX-1.5U" H 9136 11768 20  0000 C CNN
-F 2 "MX_Alps_Hybrid:MX-1.5U-Vertical" H 9025 11600 60  0001 C CNN
+F 2 "MX_Alps_Hybrid:MXOnly-1.5U-Vertical" H 9025 11600 60  0001 C CNN
 F 3 "" H 9025 11600 60  0001 C CNN
 	1    9050 11625
@@
 NoConn ~ 5800 14225
 $Comp
-L Connector_Generic:Conn_01x01 J15
-U 1 1 5BCD1D42
-P 14650 2150
-F 0 "J15" H 14729 2192 50  0000 L CNN
-F 1 "Breakaway_Tabs" H 14729 2101 50  0000 L CNN
-F 2 "locallib:breakaway-mousebites" H 14650 2150 50  0001 C CNN
-F 3 "~" H 14650 2150 50  0001 C CNN
-	1    14650 2150
-	1    0    0    -1
-$EndComp
-$Comp
 L Connector_Generic:Conn_01x01 J17
 U 1 1 5BCD1D49
@@
 NoConn ~ 5800 14750
 NoConn ~ 5800 14575
-NoConn ~ 14450 2150
 $Comp
 L Connector_Generic:Conn_01x01 J14
@@
 Connection ~ 9750 11950
 Wire Notes Line
-	14300 675  16150 675
-Wire Notes Line
-	16150 675  16150 2325
-Wire Notes Line
-	16150 2325 14300 2325
-Wire Notes Line
-	14300 2325 14300 675
-$Comp
-L Connector_Generic:Conn_01x01 J21
-U 1 1 5C31FC53
-P 14875 1050
-F 0 "J21" H 14955 1092 50  0000 L CNN
-F 1 "Conn_01x01" H 14955 1001 50  0000 L CNN
-F 2 "Mounting_Holes:MountingHole_3.5mm_Pad_Via" H 14875 1050 50  0001 C CNN
-F 3 "~" H 14875 1050 50  0001 C CNN
-	1    14875 1050
-	1    0    0    -1
-$EndComp
-Text Notes 14325 775  0    50   ~ 0
-Extras
-$Comp
-L power:GNDS #PWR01
-U 1 1 5C3200EF
-P 14675 1050
-F 0 "#PWR01" H 14675 800 50  0001 C CNN
-F 1 "GNDS" H 14680 877 50  0000 C CNN
-F 2 "" H 14675 1050 50  0001 C CNN
-F 3 "" H 14675 1050 50  0001 C CNN
-	1    14675 1050
-	1    0    0    -1
-$EndComp
-Wire Notes Line
 	9175 5250 9175 7700
 Wire Notes Line
@@
 	12025 11800 12025 12425
 Connection ~ 12025 11800
+$Comp
+L MX_Alps_Hybrids:MX-1U MXA1
+U 1 1 5D6CAD01
+P 13100 4050
+F 0 "MXA1" H 13186 4267 60  0000 C CNN
+F 1 "ALPS-1.5U" H 13186 4193 20  0000 C CNN
+F 2 "MX_Alps_Hybrid:ALPS-1.5U" H 13075 4025 60  0001 C CNN
+F 3 "" H 13075 4025 60  0001 C CNN
+	1    13100 4050
+	1    0    0    -1
+$EndComp
+$Comp
+L MX_Alps_Hybrids:MX-1U MXA2
+U 1 1 5D6CC429
+P 8575 11625
+F 0 "MXA2" H 8661 11842 60  0000 C CNN
+F 1 "ALPS-1.5U" H 8661 11768 20  0000 C CNN
+F 2 "MX_Alps_Hybrid:ALPS-1.5U" H 8550 11600 60  0001 C CNN
+F 3 "" H 8550 11600 60  0001 C CNN
+	1    8575 11625
+	1    0    0    -1
+$EndComp
+Wire Wire Line
+	9225 11600 8850 11600
+Wire Wire Line
+	8850 11600 8850 11525
+Wire Wire Line
+	8850 11525 8550 11525
+Wire Wire Line
+	8550 11525 8550 11800
+Connection ~ 9225 11600
+Wire Wire Line
+	8750 11600 8750 11800
+Wire Wire Line
+	8750 11800 8950 11800
+Connection ~ 8950 11800
+Wire Wire Line
+	12625 4225 13000 4225
+Wire Wire Line
+	13000 4225 13000 3925
+Wire Wire Line
+	13000 3925 13275 3925
+Wire Wire Line
+	13275 3925 13275 4025
+Connection ~ 12625 4225
+Wire Wire Line
+	13075 4225 13075 4025
+Wire Wire Line
+	13075 4025 12825 4025
+Connection ~ 12825 4025
 $EndSCHEMATC
