File: Orbit-Choc-PCB/Orbit.sch (KiCad schematic (older format))
At the start: 226 parts, among them J1 PJ-3200B-4A, J10 Breakaway_Tabs, J11 PJ-3200B-4A, J12 AVR-ISP-6, J13 Breakaway_Tabs, J14 Breakaway_Tabs, J17 Breakaway_Tabs, J18 Breakaway_Tabs, J19 Breakaway_Tabs, J2 AVR-ISP-6, J20 Breakaway_Tabs, J3 Breakaway_Tabs, J5 Breakaway_Tabs, J6 Breakaway_Tabs, J7 Breakaway_Tabs, J9 Breakaway_Tabs, Q1 2N7002, Q2 2N7002, SW1 SW_Push, SW2 SW_Push, U1 ATmega32U4-MU, U2 PRTR5V0U2X, U3 ATmega32U4-MU, U4 PRTR5V0U2X, Y1 16MHz, Y2 16MHz

Commit message: Build Orbit-C PCB for Choc switches
Parts:
- removed D35, D70, D71, D72, D73, D74: LED_3mm, locallib:LED_D3.0mm, symbol Device:LED_Small
- removed J1, J11: PJ-3200B-4A, locallib:PJ-3200B-4A, symbol Connector_Generic:Conn_01x04
- removed J10, J19, J20, J6: Breakaway_Tabs, locallib:breakaway-mousebites, symbol Connector_Generic:Conn_01x01
- removed MH1, MH2: HOLE, Mounting_Holes:MountingHole_5mm, symbol Connector_Generic:Conn_01x01
- removed Q1, Q2: 2N7002, TO_SOT_Packages_SMD:SOT-23, symbol Transistor_FET:2N7002
- removed R58, R60, R61, R62, R63, R64, R65, R68, R69, R70, R71, R72, R73, R75, R76, R77, R78, R79, R80: 470, Resistors_SMD:R_0805, symbol Device:R_Small
- removed R81, R82, R89, R90, R91, R92: 1k, Resistors_SMD:R_0805, symbol Device:R_Small
- added Q1, Q2: 2N7002, TO_SOT_Packages_SMD:SOT-23, symbol Device:Q_NPN_BEC
- added R1, R11, R18, R2, R26, R3, R4, R45, R46, R47, R48, R49, R5, R50, R51, R52, R6, R7, R8: 1k, Resistors_SMD:R_0805, symbol Device:R_Small
- added USB3, USB4: HRO-TYPE-C-31-M-12, Type-C:HRO-TYPE-C-31-M-13, symbol Type-C:HRO-TYPE-C-31-M-12
- J12, J2: footprint Molex-0548190589:Reset_Pretty-Mask -> random-keyboard-parts:Reset_Pretty-Mask
- MX10, MX11, MX12, MX13, MX14, MX16, MX17, MX18, MX19, MX20, MX21, MX23, MX24, MX25, MX26, MX27, MX28, MX29, MX30, MX31, MX32, MX33, MX42, MX43, MX44, MX45, MX46, MX47, MX49, MX50, MX51, MX52, MX53, MX54, MX56, MX57, MX58, MX59, MX60, MX61, MX64, MX65, MX66, MX67, MX68, MX9: footprint MX_Alps_Hybrid:MX-1U -> MX_Alps_Hybrid:KailhChoc-1U
- MX34, MX63: footprint MX_Alps_Hybrid:MXOnly-1.5U-Vertical -> MX_Alps_Hybrid:KailhChoc-1.5U
- R12, R13, R14, R15, R16, R17, R19, R20, R21, R22, R23, R24, R27, R28, R29, R30, R31, R32, R34, R35, R36, R37, R38, R39, R53, R54, R55, R56, R57: value 470 -> 1k
- SW1, SW2: footprint locallib:SKQGADE010 -> random-keyboard-parts:SKQGADE010
- U2, U4: footprint locallib:SOT143B -> random-keyboard-parts:SOT143B
- USB1, USB2: footprint Type-C:HRO-TYPE-C-31-M-12-Assembly -> Type-C:HRO-TYPE-C-31-M-13
Connections:
- net labels removed: LEDIND-1, LEDIND-1-R, LEDIND-2, LEDIND-2-R, LEDIND-3, LEDIND-3-R, LEDPWM, LEDPWM-R
- no-connect marks 20 -> 14
Other:
- note removed: "Backlight Control"
- note removed: "Indicator LEDs\n"
- note removed: "Passthrough Holes"
- note removed: "Passthrough Holes\n"
