File: Orbit-Choc-PCB/Orbit.kicad_pcb (KiCad board)
At the start: 2 copper layers, 269.5 x 125.3 mm, 1 part

Commit message: Build Orbit-C PCB for Choc switches
Parts:
- added C1: 22pF, Capacitors_SMD:C_0603, B.Cu at (107.2, 116.7)
- added C10: 1uF, Capacitors_SMD:C_0603, B.Cu at (215.9, 104.0)
- added C11: 0.1uF, Capacitors_SMD:C_0603, B.Cu at (205.6, 98.4)
- added C12: 0.1uF, Capacitors_SMD:C_0603, B.Cu at (203.2, 108.0)
- added C13: 0.1uF, Capacitors_SMD:C_0603, B.Cu at (215.9, 109.5)
- added C14: 10uF, Capacitors_SMD:C_0603, B.Cu at (211.9, 98.4)
- added C2: 22pF, Capacitors_SMD:C_0603, B.Cu at (110.7, 113.5)
- added C3: 1uF, Capacitors_SMD:C_0603, B.Cu at (114.3, 104.8)
- added C4: 0.1uF, Capacitors_SMD:C_0603, B.Cu at (114.3, 111.1)
- added C5: 0.1uF, Capacitors_SMD:C_0603, B.Cu at (100.5, 108.1)
- added C6: 0.1uF, Capacitors_SMD:C_0603, B.Cu at (103.1, 98.9)
- added C7: 10uF, Capacitors_SMD:C_0603, B.Cu at (109.7, 98.9)
- added C8: 22pF, Capacitors_SMD:C_0603, B.Cu at (209.6, 116.2)
- added C9: 22pF, Capacitors_SMD:C_0603, B.Cu at (213.2, 112.9)
- added D10: SOD-123, Diodes_SMD:D_SOD-123, B.Cu at (49.2, 54.8)
- added D11: SOD-123, Diodes_SMD:D_SOD-123, B.Cu at (68.3, 50.0)
- added D12: SOD-123, Diodes_SMD:D_SOD-123, B.Cu at (87.3, 47.6)
- added D13: SOD-123, Diodes_SMD:D_SOD-123, B.Cu at (106.4, 50.0)
- added D14: SOD-123, Diodes_SMD:D_SOD-123, B.Cu at (125.4, 52.4)
- added D16: SOD-123, Diodes_SMD:D_SOD-123, B.Cu at (30.2, 73.8)
- added D17: SOD-123, Diodes_SMD:D_SOD-123, B.Cu at (49.2, 73.8)
- added D18: SOD-123, Diodes_SMD:D_SOD-123, B.Cu at (68.3, 69.1)
- added D19: SOD-123, Diodes_SMD:D_SOD-123, B.Cu at (87.3, 66.7)
- added D20: SOD-123, Diodes_SMD:D_SOD-123, B.Cu at (106.4, 69.1)
- added D21: SOD-123, Diodes_SMD:D_SOD-123, B.Cu at (125.4, 71.4)
- added D23: SOD-123, Diodes_SMD:D_SOD-123, B.Cu at (30.2, 92.9)
- added D24: SOD-123, Diodes_SMD:D_SOD-123, B.Cu at (49.2, 92.9)
- added D25: SOD-123, Diodes_SMD:D_SOD-123, B.Cu at (68.3, 88.1)
- added D26: SOD-123, Diodes_SMD:D_SOD-123, B.Cu at (87.3, 85.7)
- added D27: SOD-123, Diodes_SMD:D_SOD-123, B.Cu at (106.4, 88.1)
- added D28: SOD-123, Diodes_SMD:D_SOD-123, B.Cu at (125.4, 90.5)
- added D29: SOD-123, Diodes_SMD:D_SOD-123, B.Cu at (30.2, 111.9)
- added D30: SOD-123, Diodes_SMD:D_SOD-123, B.Cu at (49.2, 111.9)
- added D31: SOD-123, Diodes_SMD:D_SOD-123, B.Cu at (68.3, 107.2)
- added D32: SOD-123, Diodes_SMD:D_SOD-123, B.Cu at (87.3, 104.8)
- added D33: SOD-123, Diodes_SMD:D_SOD-123, B.Cu at (126.2, 103.2)
- added D34: SOD-123, Diodes_SMD:D_SOD-123, B.Cu at (130.2, 103.2)
- added D43: SOD-123, Diodes_SMD:D_SOD-123, B.Cu at (182.6, 52.4)
- added D44: SOD-123, Diodes_SMD:D_SOD-123, B.Cu at (201.6, 50.0)
- added D45: SOD-123, Diodes_SMD:D_SOD-123, B.Cu at (220.7, 47.6)
- added D46: SOD-123, Diodes_SMD:D_SOD-123, B.Cu at (239.7, 50.0)
- added D47: SOD-123, Diodes_SMD:D_SOD-123, B.Cu at (258.8, 54.8)
- added D48: SOD-123, Diodes_SMD:D_SOD-123, B.Cu at (277.8, 54.8)
- added D50: SOD-123, Diodes_SMD:D_SOD-123, B.Cu at (182.6, 71.4)
- added D51: SOD-123, Diodes_SMD:D_SOD-123, B.Cu at (201.6, 69.1)
- added D52: SOD-123, Diodes_SMD:D_SOD-123, B.Cu at (220.7, 66.7)
- added D53: SOD-123, Diodes_SMD:D_SOD-123, B.Cu at (239.7, 69.1)
- added D54: SOD-123, Diodes_SMD:D_SOD-123, B.Cu at (258.8, 73.8)
- added D55: SOD-123, Diodes_SMD:D_SOD-123, B.Cu at (277.8, 73.8)
- added D57: SOD-123, Diodes_SMD:D_SOD-123, B.Cu at (182.6, 90.5)
- added D58: SOD-123, Diodes_SMD:D_SOD-123, B.Cu at (201.6, 88.1)
- added D59: SOD-123, Diodes_SMD:D_SOD-123, B.Cu at (220.7, 85.7)
- added D60: SOD-123, Diodes_SMD:D_SOD-123, B.Cu at (239.7, 88.1)
- added D61: SOD-123, Diodes_SMD:D_SOD-123, B.Cu at (258.8, 92.9)
- added D62: SOD-123, Diodes_SMD:D_SOD-123, B.Cu at (277.8, 92.9)
- added D64: SOD-123, Diodes_SMD:D_SOD-123, B.Cu at (176.2, 108.0)
- added D65: SOD-123, Diodes_SMD:D_SOD-123, B.Cu at (180.2, 108.0)
- added D66: SOD-123, Diodes_SMD:D_SOD-123, B.Cu at (220.7, 104.8)
- added D67: SOD-123, Diodes_SMD:D_SOD-123, B.Cu at (239.7, 107.2)
- added D68: SOD-123, Diodes_SMD:D_SOD-123, B.Cu at (258.8, 111.9)
- added D69: SOD-123, Diodes_SMD:D_SOD-123, B.Cu at (277.8, 111.9)
- added D75: Schottky, Diodes_SMD:D_SOD-123, B.Cu at (48.4, 67.5)
- added D76: Schottky, Diodes_SMD:D_SOD-123, B.Cu at (272.3, 71.4)
- added D9: SOD-123, Diodes_SMD:D_SOD-123, B.Cu at (30.2, 54.8)
- added F1: 500mA, Fuse_Holders_and_Fuses:Fuse_SMD1206_Reflow, B.Cu at (37.3, 65.1)
- added F2: 500mA, Fuse_Holders_and_Fuses:Fuse_SMD1206_Reflow, B.Cu at (277.0, 65.1)
- added FID1: Fiducial, Fiducials:Fiducial_1mm_Dia_2.54mm_Outer_CopperTop, B.Cu at (25.4, 27.8)
- added FID2: Fiducial, Fiducials:Fiducial_1mm_Dia_2.54mm_Outer_CopperTop, B.Cu at (288.9, 27.8)
- added FID3: Fiducial, Fiducials:Fiducial_1mm_Dia_2.54mm_Outer_CopperTop, B.Cu at (288.9, 146.8)
- added FID4: Fiducial, Fiducials:Fiducial_1mm_Dia_2.54mm_Outer_CopperTop, F.Cu at (25.4, 27.8)
- added FID5: Fiducial, Fiducials:Fiducial_1mm_Dia_2.54mm_Outer_CopperTop, F.Cu at (288.9, 27.8)
- added FID6: Fiducial, Fiducials:Fiducial_1mm_Dia_2.54mm_Outer_CopperTop, F.Cu at (288.9, 146.8)
- added G***: LOGO, locallib:ai-ring-6mm, F.Cu at (37.3, 138.9)
- added G***: LOGO, locallib:ai-ring-6mm-Combined, B.Cu at (175.4, 129.4)
- added G***: LOGO, locallib:ai-ring-6mm-Combined, B.Cu at (138.9, 130.2)
- added G***: LOGO, locallib:ai-ring-6mm-FancyAss, F.Cu at (138.9, 130.2)
- added G***: LOGO, locallib:ai-ring-6mm-FancyAss, F.Cu at (175.4, 129.4)
- added J12: AVR-ISP-6, random-keyboard-parts:Reset_Pretty-Mask, B.Cu at (187.3, 119.9)
- added J13: Breakaway_Tabs, locallib:breakaway-mousebites, B.Cu at (71.4, 39.7)
- added J14: Breakaway_Tabs, locallib:breakaway-mousebites, B.Cu at (81.0, 119.1)
- added J17: Breakaway_Tabs, locallib:breakaway-mousebites, B.Cu at (42.9, 122.7)
- added J18: Breakaway_Tabs, locallib:breakaway-mousebites, B.Cu at (81.0, 122.7)
- added J2: AVR-ISP-6, random-keyboard-parts:Reset_Pretty-Mask, B.Cu at (127.0, 118.3)
- added J3: Breakaway_Tabs, locallib:breakaway-mousebites, B.Cu at (271.3, 122.7)
- added J5: Breakaway_Tabs, locallib:breakaway-mousebites, B.Cu at (233.2, 119.1)
- added J7: Breakaway_Tabs, locallib:breakaway-mousebites, B.Cu at (242.7, 39.7)
- added J9: Breakaway_Tabs, locallib:breakaway-mousebites, B.Cu at (233.2, 122.7)
- added MX10: MX-1U, MX_Alps_Hybrid:KailhChoc-1U, F.Cu at (52.4, 55.6)
- added MX11: MX-1U, MX_Alps_Hybrid:KailhChoc-1U, F.Cu at (71.4, 50.8)
- added MX12: MX-1U, MX_Alps_Hybrid:KailhChoc-1U, F.Cu at (90.5, 48.4)
- added MX13: MX-1U, MX_Alps_Hybrid:KailhChoc-1U, F.Cu at (109.5, 50.8)
- added MX14: MX-1U, MX_Alps_Hybrid:KailhChoc-1U, F.Cu at (128.6, 53.2)
- added MX16: MX-1U, MX_Alps_Hybrid:KailhChoc-1U, F.Cu at (33.3, 74.6)
- added MX17: MX-1U, MX_Alps_Hybrid:KailhChoc-1U, F.Cu at (52.4, 74.6)
- added MX18: MX-1U, MX_Alps_Hybrid:KailhChoc-1U, F.Cu at (71.4, 69.8)
- added MX19: MX-1U, MX_Alps_Hybrid:KailhChoc-1U, F.Cu at (90.5, 67.5)
- added MX20: MX-1U, MX_Alps_Hybrid:KailhChoc-1U, F.Cu at (109.5, 69.8)
- added MX21: MX-1U, MX_Alps_Hybrid:KailhChoc-1U, F.Cu at (128.6, 72.2)
- added MX23: MX-1U, MX_Alps_Hybrid:KailhChoc-1U, F.Cu at (33.3, 93.7)
- added MX24: MX-1U, MX_Alps_Hybrid:KailhChoc-1U, F.Cu at (52.4, 93.7)
- added MX25: MX-1U, MX_Alps_Hybrid:KailhChoc-1U, F.Cu at (71.4, 88.9)
- added MX26: MX-1U, MX_Alps_Hybrid:KailhChoc-1U, F.Cu at (90.5, 86.5)
- added MX27: MX-1U, MX_Alps_Hybrid:KailhChoc-1U, F.Cu at (109.5, 88.9)
- added MX28: MX-1U, MX_Alps_Hybrid:KailhChoc-1U, F.Cu at (128.6, 91.3)
- added MX29: MX-1U, MX_Alps_Hybrid:KailhChoc-1U, F.Cu at (33.3, 112.7)
- added MX30: MX-1U, MX_Alps_Hybrid:KailhChoc-1U, F.Cu at (52.4, 112.7)
- added MX31: MX-1U, MX_Alps_Hybrid:KailhChoc-1U, F.Cu at (71.4, 108.0)
- added MX32: MX-1U, MX_Alps_Hybrid:KailhChoc-1U, F.Cu at (90.5, 105.6)
- added MX33: MX-1U, MX_Alps_Hybrid:KailhChoc-1U, F.Cu at (119.1, 110.9)
- added MX34: MX-1.5U, MX_Alps_Hybrid:KailhChoc-1.5U, F.Cu at (139.2, 118.2)
- added MX42: MX-1U, MX_Alps_Hybrid:KailhChoc-1U, F.Cu at (185.6, 53.2)
- added MX43: MX-1U, MX_Alps_Hybrid:KailhChoc-1U, F.Cu at (204.6, 50.8)
- added MX44: MX-1U, MX_Alps_Hybrid:KailhChoc-1U, F.Cu at (223.7, 48.4)
- added MX45: MX-1U, MX_Alps_Hybrid:KailhChoc-1U, F.Cu at (242.7, 50.8)
- added MX46: MX-1U, MX_Alps_Hybrid:KailhChoc-1U, F.Cu at (261.8, 55.6)
- added MX47: MX-1U, MX_Alps_Hybrid:KailhChoc-1U, F.Cu at (280.8, 55.6)
- added MX49: MX-1U, MX_Alps_Hybrid:KailhChoc-1U, F.Cu at (185.6, 72.2)
- added MX50: MX-1U, MX_Alps_Hybrid:KailhChoc-1U, F.Cu at (204.6, 69.8)
- added MX51: MX-1U, MX_Alps_Hybrid:KailhChoc-1U, F.Cu at (223.7, 67.5)
- added MX52: MX-1U, MX_Alps_Hybrid:KailhChoc-1U, F.Cu at (242.7, 69.8)
- added MX53: MX-1U, MX_Alps_Hybrid:KailhChoc-1U, F.Cu at (261.8, 74.6)
- added MX54: MX-1U, MX_Alps_Hybrid:KailhChoc-1U, F.Cu at (280.8, 74.6)
- added MX56: MX-1U, MX_Alps_Hybrid:KailhChoc-1U, F.Cu at (185.6, 91.3)
- added MX57: MX-1U, MX_Alps_Hybrid:KailhChoc-1U, F.Cu at (204.6, 88.9)
- added MX58: MX-1U, MX_Alps_Hybrid:KailhChoc-1U, F.Cu at (223.7, 86.5)
- added MX59: MX-1U, MX_Alps_Hybrid:KailhChoc-1U, F.Cu at (242.7, 88.9)
- added MX60: MX-1U, MX_Alps_Hybrid:KailhChoc-1U, F.Cu at (261.8, 93.7)
- added MX61: MX-1U, MX_Alps_Hybrid:KailhChoc-1U, F.Cu at (280.8, 93.7)
- added MX63: MX-1.5U, MX_Alps_Hybrid:KailhChoc-1.5U, F.Cu at (175.0, 118.2)
- added MX64: MX-1U, MX_Alps_Hybrid:KailhChoc-1U, F.Cu at (195.0, 110.9)
- added MX65: MX-1U, MX_Alps_Hybrid:KailhChoc-1U, F.Cu at (223.7, 105.6)
- added MX66: MX-1U, MX_Alps_Hybrid:KailhChoc-1U, F.Cu at (242.7, 108.0)
- added MX67: MX-1U, MX_Alps_Hybrid:KailhChoc-1U, F.Cu at (261.8, 112.7)
- added MX68: MX-1U, MX_Alps_Hybrid:KailhChoc-1U, F.Cu at (280.8, 112.7)
- added MX9: MX-1U, MX_Alps_Hybrid:KailhChoc-1U, F.Cu at (33.3, 55.6)
- added Q1: 2N7002, TO_SOT_Packages_SMD:SOT-23, B.Cu at (133.3, 108.7)
- added Q2: 2N7002, TO_SOT_Packages_SMD:SOT-23, B.Cu at (234.2, 102.4)
- added R1: 1k, Resistors_SMD:R_0805, B.Cu at (129.4, 108.7)
- added R10: 4.7k, Resistors_SMD:R_0805, B.Cu at (122.2, 98.6)
- added R11: 1k, Resistors_SMD:R_0805, B.Cu at (57.9, 78.6)
- added R12: 1k, Resistors_SMD:R_0805, B.Cu at (77.0, 73.8)
- added R13: 1k, Resistors_SMD:R_0805, B.Cu at (96.0, 71.4)
- added R14: 1k, Resistors_SMD:R_0805, B.Cu at (115.1, 73.8)
- added R15: 1k, Resistors_SMD:R_0805, B.Cu at (134.1, 76.2)
- added R16: 1k, Resistors_SMD:R_0805, B.Cu at (38.9, 97.6)
- added R17: 1k, Resistors_SMD:R_0805, B.Cu at (57.9, 97.6)
- added R18: 1k, Resistors_SMD:R_0805, B.Cu at (77.0, 92.9)
- added R19: 1k, Resistors_SMD:R_0805, B.Cu at (96.0, 90.5)
- added R2: 1k, Resistors_SMD:R_0805, B.Cu at (38.9, 59.5)
- added R20: 1k, Resistors_SMD:R_0805, B.Cu at (115.1, 92.9)
- added R21: 1k, Resistors_SMD:R_0805, B.Cu at (131.8, 91.3)
- added R22: 1k, Resistors_SMD:R_0805, B.Cu at (38.9, 116.7)
- added R23: 1k, Resistors_SMD:R_0805, B.Cu at (57.9, 116.7)
- added R24: 1k, Resistors_SMD:R_0805, B.Cu at (77.0, 111.9)
- added R25: 10k, Resistors_SMD:R_0805, B.Cu at (97.6, 112.7)
- added R26: 1k, Resistors_SMD:R_0805, B.Cu at (83.3, 109.5)
- added R27: 1k, Resistors_SMD:R_0805, B.Cu at (122.0, 120.7)
- added R28: 1k, Resistors_SMD:R_0805, B.Cu at (135.7, 119.9)
- added R29: 1k, Resistors_SMD:R_0805, B.Cu at (234.2, 106.4)
- added R3: 1k, Resistors_SMD:R_0805, B.Cu at (57.9, 59.5)
- added R30: 1k, Resistors_SMD:R_0805, B.Cu at (178.6, 57.1)
- added R31: 1k, Resistors_SMD:R_0805, B.Cu at (210.3, 54.8)
- added R32: 1k, Resistors_SMD:R_0805, B.Cu at (229.4, 52.4)
- added R33: 1k, Resistors_SMD:R_0805, B.Cu at (248.4, 54.8)
- added R34: 1k, Resistors_SMD:R_0805, B.Cu at (254.0, 59.5)
- added R35: 1k, Resistors_SMD:R_0805, B.Cu at (286.5, 59.5)
- added R36: 1k, Resistors_SMD:R_0805, B.Cu at (191.3, 76.2)
- added R37: 1k, Resistors_SMD:R_0805, B.Cu at (210.3, 73.8)
- added R38: 1k, Resistors_SMD:R_0805, B.Cu at (229.4, 71.4)
- added R39: 1k, Resistors_SMD:R_0805, B.Cu at (248.4, 73.8)
- added R4: 1k, Resistors_SMD:R_0805, B.Cu at (77.0, 54.8)
- added R40: 1k, Resistors_SMD:R_0805, B.Cu at (267.5, 78.6)
- added R41: 22, Resistors_SMD:R_0805, B.Cu at (63.5, 59.5)
- added R42: 22, Resistors_SMD:R_0805, B.Cu at (63.5, 62.7)
- added R43: 5.1k, Resistors_SMD:R_0805, B.Cu at (57.1, 47.6)
- added R44: 5.1k, Resistors_SMD:R_0805, B.Cu at (29.4, 49.2)
- added R45: 1k, Resistors_SMD:R_0805, B.Cu at (286.5, 78.6)
- added R46: 1k, Resistors_SMD:R_0805, B.Cu at (191.3, 95.2)
- added R47: 1k, Resistors_SMD:R_0805, B.Cu at (210.3, 92.9)
- added R48: 1k, Resistors_SMD:R_0805, B.Cu at (229.4, 90.5)
- added R49: 1k, Resistors_SMD:R_0805, B.Cu at (248.4, 92.9)
- added R5: 1k, Resistors_SMD:R_0805, B.Cu at (96.0, 52.4)
- added R50: 1k, Resistors_SMD:R_0805, B.Cu at (267.5, 97.6)
- added R51: 1k, Resistors_SMD:R_0805, B.Cu at (286.5, 97.6)
- added R52: 1k, Resistors_SMD:R_0805, B.Cu at (176.2, 113.5)
- added R53: 1k, Resistors_SMD:R_0805, B.Cu at (184.2, 113.5)
- added R54: 1k, Resistors_SMD:R_0805, B.Cu at (229.4, 109.5)
- added R55: 1k, Resistors_SMD:R_0805, B.Cu at (248.4, 111.9)
- added R56: 1k, Resistors_SMD:R_0805, B.Cu at (267.5, 116.7)
- added R57: 1k, Resistors_SMD:R_0805, B.Cu at (286.5, 116.7)
- added R6: 1k, Resistors_SMD:R_0805, B.Cu at (115.1, 54.8)
- added R67: 10k, Resistors_SMD:R_0805, B.Cu at (201.6, 115.1)
- added R7: 1k, Resistors_SMD:R_0805, B.Cu at (134.1, 57.1)
- added R8: 1k, Resistors_SMD:R_0805, B.Cu at (38.9, 78.6)
- added R83: 22, Resistors_SMD:R_0805, B.Cu at (254.8, 66.7)
- added R84: 22, Resistors_SMD:R_0805, B.Cu at (254.8, 63.5)
- added R85: 5.1k, Resistors_SMD:R_0805, B.Cu at (285.8, 47.6)
- added R86: 5.1k, Resistors_SMD:R_0805, B.Cu at (257.2, 48.4)
- added R87: 10k, Resistors_SMD:R_0805, B.Cu at (100.8, 112.7)
- added R88: 10k, Resistors_SMD:R_0805, B.Cu at (204.0, 115.1)
- added R9: 4.7k, Resistors_SMD:R_0805, B.Cu at (122.2, 101.6)
- added SW1: SW_Push, random-keyboard-parts:SKQGADE010, B.Cu at (135.7, 101.6)
- added SW2: SW_Push, random-keyboard-parts:SKQGADE010, B.Cu at (185.7, 106.4)
- added U1: ATmega32U4-MU, Housings_DFN_QFN:QFN-44-1EP_7x7mm_Pitch0.5mm, B.Cu at (106.4, 104.8)
- added U2: PRTR5V0U2X, random-keyboard-parts:SOT143B, B.Cu at (42.9, 53.2)
- added U3: ATmega32U4-MU, Housings_DFN_QFN:QFN-44-1EP_7x7mm_Pitch0.5mm, B.Cu at (208.9, 104.5)
- added U4: PRTR5V0U2X, random-keyboard-parts:SOT143B, B.Cu at (271.5, 53.2)
- added USB1: HRO-TYPE-C-31-M-12, Type-C:HRO-TYPE-C-31-M-13, B.Cu at (42.9, 40.3)
- added USB2: HRO-TYPE-C-31-M-12, Type-C:HRO-TYPE-C-31-M-13, B.Cu at (271.3, 40.3)
- added USB3: HRO-TYPE-C-31-M-12, Type-C:HRO-TYPE-C-31-M-13, B.Cu at (119.1, 36.4)
- added USB4: HRO-TYPE-C-31-M-12, Type-C:HRO-TYPE-C-31-M-13, B.Cu at (195.1, 36.4)
- added Y1: 16MHz, Crystals:Crystal_SMD_3225-4pin_3.2x2.5mm, B.Cu at (107.2, 113.5)
- added Y2: 16MHz, Crystals:Crystal_SMD_3225-4pin_3.2x2.5mm, B.Cu at (209.6, 112.9)
- moved REF** 1.84 mm to (22.3, 149.7)
Routing:
- net +5V: track 0.00 -> 730.3 mm, vias 0 -> 11
- net +5VA: track 0.00 -> 699.8 mm, vias 0 -> 9
- net LEDGND-R: track 0.00 -> 462.1 mm, vias 0 -> 13
- net LEDGND: track 0.00 -> 459.2 mm, vias 0 -> 13
- net GND: track 0.00 -> 394.4 mm, vias 0 -> 8
- net GNDA: track 0.00 -> 385.5 mm, vias 0 -> 4
- net ROW3-R: track 0.00 -> 180.0 mm, vias 0 -> 7
- net ROW0-R: track 0.00 -> 164.7 mm, vias 0 -> 6
- net ROW0: track 0.00 -> 159.6 mm, vias 0 -> 6
- net COL5-R: track 0.00 -> 149.3 mm
- net ROW1-R: track 0.00 -> 144.7 mm, vias 0 -> 2
- net ROW1: track 0.00 -> 140.5 mm, vias 0 -> 2
- net COL0: track 0.00 -> 133.5 mm
- net VBUS: track 0.00 -> 131.9 mm, vias 0 -> 4
- net COL4-R: track 0.00 -> 127.6 mm
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- added copper zone on B.Cu, net GND
- added copper zone on B.Cu, net GNDA
Other:
- outline, holes or cut-outs redrawn
- board text added: "Orbit-C PCB R1.0"
- board text added: "Orbit-C PCB Rev 1.0 20190130"
- board text added: "kb.ai03.me"

Commit message: Update traces
Routing:
- net COL5: track 98.6 -> 99.4 mm
Other:
- board text added: "I2C"
- board text added: "USB"
