File: OrbitX-PCB/Orbit.kicad_pcb (KiCad board)
At the start: 2 copper layers, 303.2 x 145.3 mm, 301 parts, among them J1 PJ-3200B-4A, J10 Breakaway_Tabs, J11 PJ-3200B-4A, J12 AVR-ISP-6, J13 Breakaway_Tabs, J14 Breakaway_Tabs, J17 Breakaway_Tabs, J18 Breakaway_Tabs, J19 Breakaway_Tabs, J2 AVR-ISP-6, J20 Breakaway_Tabs, J3 Breakaway_Tabs, J5 Breakaway_Tabs, J6 Breakaway_Tabs, J7 Breakaway_Tabs, J9 Breakaway_Tabs, Q1 2N7002, Q2 2N7002, SW1 SW_Push, SW2 SW_Push, U1 ATmega32U4-MU, U2 PRTR5V0U2X, U3 ATmega32U4-MU, U4 PRTR5V0U2X, Y1 16MHz, Y2 16MHz

Commit message: Place switches, draw outline
Parts:
- removed D49, D50, D51, D52, D53, D54, D55, D56, D57, D58, D59, D60, D61, D62, D63, D64, D65, D66, D67, D68, D69: SOD-123, Diodes_SMD:D_SOD-123
- removed D70, D71, D72, D73, D74: LED_3mm, locallib:LED_D3.0mm
- removed G*** (x2): LOGO, locallib:Orbit
- removed G***: LOGO, locallib:ai-outline-7.6
- removed G*** (x2): LOGO, locallib:ai-ring-6mm-FancyAss
- removed G*** (x2): LOGO, locallib:ai-ring-6mm-Combined
- removed MH1, MH2: HOLE, Mounting_Holes:MountingHole_5mm
- removed MX49, MX50, MX51, MX52, MX53, MX54, MX55, MX56, MX57, MX58, MX59, MX60, MX61, MX62, MX64, MX65, MX66, MX67, MX68: MX-1U, MX_Alps_Hybrid:MX-1U
- removed MX63: MX-1.5U, MX_Alps_Hybrid:MXOnly-1.5U-Vertical
- removed MXA1, MXA2: ALPS-1.5U, MX_Alps_Hybrid:ALPS-1.5U
- removed MXE-1, MXE-2: MX-2U, MX_Alps_Hybrid:MX-2U
- removed MXE-3, MXE-4, MXE-5, MXE-6: MX-2U, MX_Alps_Hybrid:MX-2U-ReversedStabilizers
- removed Q1, Q2: 2N7002, TO_SOT_Packages_SMD:SOT-23
- removed R11, R12, R13, R14, R15, R16, R17, R18, R19, R2, R20, R21, R22, R23, R24, R26, R27, R28, R29, R3, R30, R31, R32, R34, R35, R36, R37, R38, R39, R4, R46, R47, R48, R49, R5, R50, R51, R52, R53, R54, R55, R56, R57, R58, R59, R6, R60, R61, R62, R63, R64, R65, R66, R68, R69, R7, R70, R71, R72, R73, R74, R75, R76, R77, R78, R79, R8, R80: 470, Resistors_SMD:R_0805
- removed R33, R40, R81, R82, R89, R90, R91, R92: 1k, Resistors_SMD:R_0805
- C1, C10, C11, C12, C13, C14, C2, C3, C4, C5, C6, C7, C8, C9: footprint Capacitors_SMD:C_0603 -> Capacitor_SMD:C_0603_1608Metric
- D1, D10, D11, D12, D13, D14, D15, D16, D17, D18, D19, D2, D20, D21, D22, D23, D24, D25, D26, D27, D28, D29, D3, D30, D31, D32, D33, D34, D36, D37, D38, D39, D4, D40, D41, D42, D43, D44, D45, D46, D47, D48, D5, D6, D7, D8, D9: value SOD-123 -> SOD123; footprint Diodes_SMD:D_SOD-123 -> Diode_SMD:D_SOD-123
- D35: value LED_3mm -> SOD123; footprint locallib:LED_D3.0mm -> Diode_SMD:D_SOD-123; moved to B.Cu
- D75, D76: footprint Diodes_SMD:D_SOD-123 -> Diode_SMD:D_SOD-123
- F1, F2: footprint Fuse_Holders_and_Fuses:Fuse_SMD1206_Reflow -> Fuse:Fuse_1206_3216Metric
- FID1, FID2, FID3: footprint Fiducials:Fiducial_1mm_Dia_2.54mm_Outer_CopperTop -> Fiducial:Fiducial_1mm_Dia_2.54mm_Outer_CopperTop; moved to B.Cu
- FID4, FID5, FID6: footprint Fiducials:Fiducial_1mm_Dia_2.54mm_Outer_CopperTop -> Fiducial:Fiducial_1mm_Dia_2.54mm_Outer_CopperTop
- J10, J13, J14, J17, J18, J19, J20, J3, J5, J6, J7, J9: moved to B.Cu
- J12, J2: footprint Molex-0548190589:Reset_Pretty-Mask -> random-keyboard-parts:Reset_Pretty-Mask
- MX1, MX10, MX11, MX13, MX14, MX15, MX16, MX17, MX18, MX19, MX2, MX20, MX21, MX22, MX23, MX24, MX25, MX26, MX27, MX28, MX29, MX3, MX30, MX31, MX32, MX33, MX35, MX36, MX37, MX38, MX39, MX4, MX41, MX42, MX43, MX44, MX45, MX46, MX47, MX48, MX5, MX6, MX7, MX8, MX9: value MX-1U -> MX-NoLED; footprint MX_Alps_Hybrid:MX-1U -> MX_Alps_Hybrid:MX-1U-NoLED
- MX12, MX40: value MX-1U -> MX-NoLED; footprint MX_Alps_Hybrid:MX-1U -> MX_Alps_Hybrid:MX-1.5U-NoLED
- MX34: value MX-1.5U -> MX-NoLED; footprint MX_Alps_Hybrid:MXOnly-1.5U-Vertical -> MX_Alps_Hybrid:MX-1U-NoLED
- R10, R25, R41, R42, R43, R44, R67, R83, R84, R85, R86, R87, R88, R9: footprint Resistors_SMD:R_0805 -> Resistor_SMD:R_0603_1608Metric
- U1, U3: footprint Housings_DFN_QFN:QFN-44-1EP_7x7mm_Pitch0.5mm -> Package_DFN_QFN:QFN-44-1EP_7x7mm_P0.5mm_EP5.2x5.2mm
- Y1, Y2: footprint Crystals:Crystal_SMD_3225-4pin_3.2x2.5mm -> Crystal:Crystal_SMD_3225-4Pin_3.2x2.5mm
- moved J13 327.1 mm to (23.7, -89.6), turned to 0 degrees
- moved J20 326.6 mm to (64.0, -72.5)
- moved J14 317.1 mm to (30.6, -89.6), turned to 0 degrees
- moved FID3 307.4 mm to (264.2, -45.7)
- moved FID6 306.2 mm to (266.2, -41.5)
- moved D48 293.5 mm to (58.6, -83.9), turned to 0 degrees
- moved D47 286.1 mm to (50.2, -87.3), turned to 0 degrees
- moved J18 276.3 mm to (57.2, -76.3)
- moved D42 271.4 mm to (77.0, -76.4), turned to 0 degrees
- moved D41 270.1 mm to (71.2, -79.7), turned to 0 degrees
- moved D46 262.7 mm to (55.9, -87.3), turned to 0 degrees
- moved SW2 251.5 mm to (39.5, -81.8), turned to 0 degrees
- moved D40 249.5 mm to (77.0, -79.7), turned to 0 degrees
- moved FID1 244.9 mm to (270.3, -42.7)
- moved FID4 244.2 mm to (270.6, -38.6)
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Connections:
- D10 pad 1: ROW1 -> ROW1-R
- D11 pad 1: ROW1 -> ROW2-R
- D12 pad 1: ROW1 -> ROW3-R
- D13 pad 1: ROW1 -> ROW0
- D16 pad 1: ROW2 -> ROW3
- D17 pad 1: ROW2 -> ROW0-R
- D18 pad 1: ROW2 -> ROW1-R
- D19 pad 1: ROW2 -> ROW2-R
- D2 pad 1: ROW0 -> ROW1
- D20 pad 1: ROW2 -> ROW3-R
- D21 pad 1: ROW2 -> ROW0
- D22 pad 1: ROW3 -> ROW1
- D23 pad 1: ROW3 -> ROW2
- D25 pad 1: ROW3 -> ROW0-R
- D26 pad 1: ROW3 -> ROW1-R
- D27 pad 1: ROW3 -> ROW2-R
- D28 pad 1: ROW3 -> ROW3-R
- D29 pad 1: ROW4 -> ROW0
- D3 pad 1: ROW0 -> ROW2
- D30 pad 1: ROW4 -> ROW1
- D31 pad 1: ROW4 -> ROW2
- D32 pad 1: ROW4 -> ROW3
- D33 pad 1: ROW4 -> ROW0-R
- D34 pad 1: ROW4 -> ROW1-R
- D35 pad 1: GND -> ROW2-R
- D36 pad 1: ROW0-R -> ROW3-R
- D37 pad 1: ROW0-R -> ROW0
- D38 pad 1: ROW0-R -> ROW1
- D39 pad 1: ROW0-R -> ROW2
- D4 pad 1: ROW0 -> ROW3
- D40 pad 1: ROW0-R -> ROW3
- D42 pad 1: ROW0-R -> ROW1-R
- D43 pad 1: ROW1-R -> ROW2-R
- D44 pad 1: ROW1-R -> ROW3-R
- D45 pad 1: ROW1-R -> ROW0-R
- D47 pad 1: ROW1-R -> ROW2-R
- D48 pad 1: ROW1-R -> ROW3-R
- D6 pad 1: ROW0 -> ROW1
- D7 pad 1: ROW0 -> ROW2
- D8 pad 1: ROW1 -> ROW3
- D9 pad 1: ROW1 -> ROW0-R
- MX10 pad 1: COL2 -> COL0-R
- MX11 pad 1: COL3 -> COL0-R
- MX12 pad 1: COL4 -> COL0-R
- MX13 pad 1: COL5 -> COL2
- MX14 pad 1: COL6 -> COL2
- MX15 pad 1: COL0 -> COL2
- MX16 pad 1: COL1 -> COL2
- MX17 pad 1: COL2 -> COL1-R
- MX18 pad 1: COL3 -> COL1-R
- MX19 pad 1: COL4 -> COL1-R
- MX2 pad 1: COL1 -> COL0
- MX20 pad 1: COL5 -> COL1-R
- MX21 pad 1: COL6 -> COL3
- MX22 pad 1: COL0 -> COL3
- MX23 pad 1: COL1 -> COL3
- MX24 pad 1: COL2 -> COL3
- MX25 pad 1: COL3 -> COL2-R
- MX26 pad 1: COL4 -> COL2-R
- MX27 pad 1: COL5 -> COL2-R
- MX28 pad 1: COL6 -> COL2-R
- MX29 pad 1: COL1 -> COL4
- MX3 pad 1: COL2 -> COL0
- MX30 pad 1: COL2 -> COL4
- MX31 pad 1: COL3 -> COL4
- MX33 pad 1: COL5 -> COL3-R
- MX34 pad 1: COL6 -> COL3-R
- MX35 pad 1: COL0-R -> COL3-R
- MX35 pad 2: Net-(D36-Pad2) -> Net-(D35-Pad2)
- MX36 pad 1: COL1-R -> COL3-R
- MX36 pad 2: Net-(D37-Pad2) -> Net-(D36-Pad2)
- MX37 pad 1: COL2-R -> COL5
- MX37 pad 2: Net-(D38-Pad2) -> Net-(D37-Pad2)
- MX38 pad 1: COL3-R -> COL5
- MX38 pad 2: Net-(D39-Pad2) -> Net-(D38-Pad2)
- MX39 pad 1: COL4-R -> COL5
- MX39 pad 2: Net-(D40-Pad2) -> Net-(D39-Pad2)
- MX4 pad 1: COL3 -> COL0
- MX40 pad 1: COL5-R -> COL5
- MX40 pad 2: Net-(D41-Pad2) -> Net-(D40-Pad2)
- MX41 pad 1: COL6-R -> COL4-R
- MX41 pad 2: Net-(D42-Pad2) -> Net-(D41-Pad2)
- MX42 pad 1: COL0-R -> COL4-R
- MX42 pad 2: Net-(D43-Pad2) -> Net-(D42-Pad2)
- MX43 pad 1: COL1-R -> COL4-R
- MX43 pad 2: Net-(D44-Pad2) -> Net-(D43-Pad2)
- MX44 pad 1: COL2-R -> COL4-R
- MX44 pad 2: Net-(D45-Pad2) -> Net-(D44-Pad2)
- MX45 pad 1: COL3-R -> COL5-R
- MX45 pad 2: Net-(D46-Pad2) -> Net-(D45-Pad2)
- MX46 pad 1: COL4-R -> COL5-R
- MX46 pad 2: Net-(D47-Pad2) -> Net-(D46-Pad2)
- MX47 pad 2: Net-(D48-Pad2) -> Net-(D47-Pad2)
- MX48 pad 1: COL6-R -> COL5-R
- MX48 pad 2: Net-(D49-Pad2) -> Net-(D48-Pad2)
- MX5 pad 1: COL4 -> COL1
- MX6 pad 1: COL5 -> COL1
- MX7 pad 1: COL6 -> COL1
- MX8 pad 1: COL0 -> COL1
- MX9 pad 1: COL1 -> COL0-R
- Y1 pad 2: GND -> Net-(Y1-Pad2)
- Y1 pad 4: GND -> Net-(Y1-Pad4)
- Y2 pad 2: GNDA -> Net-(Y2-Pad2)
- Y2 pad 4: GNDA -> Net-(Y2-Pad4)
Routing:
- net +5V: track 980.7 -> 0.00 mm, vias 14 -> 0
- net +5VA: track 945.4 -> 0.00 mm, vias 13 -> 0
- net LEDGND-R: track 681.7 -> 0.00 mm, vias 19 -> 0
- net LEDGND: track 666.3 -> 0.00 mm, vias 17 -> 0
- net GND: track 540.0 -> 42.1 mm, vias 5 -> 0
- net GNDA: track 510.4 -> 51.2 mm, vias 6 -> 0
- net ROW0-R: track 205.8 -> 0.00 mm, vias 4 -> 0
- net ROW0: track 196.3 -> 0.00 mm, vias 4 -> 0
- net ROW1-R: track 177.0 -> 0.00 mm, vias 4 -> 0
- net ROW1: track 173.1 -> 0.00 mm, vias 4 -> 0
- net COL0: track 167.9 -> 0.00 mm
- net COL1: track 163.0 -> 0.00 mm
- net ROW2-R: track 159.8 -> 0.00 mm, vias 4 -> 0
- net ROW2: track 155.7 -> 0.00 mm, vias 4 -> 0
- net COL5-R: track 150.8 -> 0.00 mm
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- removed copper zone on B.Cu, net GND
- removed copper zone on B.Cu, net GNDA
Other:
- board size 303.2 x 145.3 mm -> 261.9 x 94.3 mm
- board text removed: "L"
- board text removed: "Orbit PCB R2.2 by ai03"
- board text removed: "Orbit PCB Revision 2.2 20181211"
- board text removed: "R"
- board text removed: "RESET"

Commit message: Progress
Parts:
- moved D44 296.1 mm to (274.6, 106.4), turned to 90 degrees
- moved D48 290.3 mm to (277.8, 106.4), turned to 90 degrees
- moved D47 286.9 mm to (277.8, 87.3), turned to 90 degrees
- moved D46 271.0 mm to (277.8, 68.3), turned to 90 degrees
- moved D43 269.5 mm to (274.6, 87.3), turned to 90 degrees
- moved D45 255.6 mm to (277.8, 49.2), turned to 90 degrees
- moved D36 251.1 mm to (239.7, 99.2), turned to 90 degrees
- moved D42 244.9 mm to (274.6, 68.3), turned to 90 degrees
- moved D41 240.8 mm to (274.6, 49.2), turned to 90 degrees
- moved D35 235.5 mm to (239.7, 80.2), turned to 90 degrees
- moved SW2 234.9 mm to (200.0, 89.7)
- moved D28 229.7 mm to (236.5, 99.2), turned to 90 degrees
- moved D20 223.6 mm to (190.5, 98.4), turned to 90 degrees
- moved D27 221.9 mm to (236.5, 80.2), turned to 90 degrees
- moved C3 220.5 mm to (104.0, 95.2), turned to 180 degrees
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Connections:
- Y1 pad 2: Net-(Y1-Pad2) -> GND
- Y1 pad 4: Net-(Y1-Pad4) -> GND
- Y2 pad 2: Net-(Y2-Pad2) -> GNDA
- Y2 pad 4: Net-(Y2-Pad4) -> GNDA
Routing:
- net GND: track 42.1 -> 148.3 mm, vias 0 -> 2
- net ROW3: track 0.00 -> 97.4 mm
- net ROW2: track 0.00 -> 93.5 mm, vias 0 -> 2
- net VBUS: track 0.00 -> 89.1 mm, vias 0 -> 3
- net ROW1-R: track 0.00 -> 87.5 mm, vias 0 -> 2
- net ROW1: track 0.00 -> 85.8 mm, vias 0 -> 4
- net ROW2-R: track 0.00 -> 83.3 mm, vias 0 -> 2
- net ROW0: track 0.00 -> 83.3 mm, vias 0 -> 4
- net ROW0-R: track 0.00 -> 83.3 mm, vias 0 -> 2
- net +5V: track 0.00 -> 76.0 mm, vias 0 -> 8
- net SCL: track 0.00 -> 71.6 mm
- net COL5: track 0.00 -> 71.5 mm
- net Net-(R41-Pad2): track 17.6 -> 88.4 mm
- net Net-(R83-Pad2): track 14.7 -> 84.3 mm
- net Net-(R42-Pad2): track 17.0 -> 86.3 mm
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Other:
- board size 261.9 x 94.3 mm -> 261.9 x 94.9 mm
- net class POWER: trace_width 0.381 -> 0.254

Commit message: Generate gerbers
Parts:
- removed FID4, FID5, FID6: Fiducial, Fiducial:Fiducial_1mm_Dia_2.54mm_Outer_CopperTop
- removed J10, J20: Breakaway_Tabs, locallib:breakaway-mousebites
- added G***: LOGO, locallib:ai-4.8-mask, F.Cu at (288.9, 130.2)
- added G***: LOGO, locallib:orbitx, F.Cu at (52.4, 95.2)
- added G***: LOGO, locallib:orbitx, F.Cu at (43.7, 130.2)
- added G***: LOGO, locallib:ai-4.8-mask, B.Cu at (144.5, 118.3)
- added G***: LOGO, locallib:ai-4.8-mask, B.Cu at (181.0, 118.3)
- added G***: LOGO, locallib:orbitx, B.Cu at (272.3, 95.2)
- added G***: LOGO, locallib:orbitx, B.Cu at (51.6, 95.2)
- added G***: LOGO, locallib:ai-4.8-mask, F.Cu at (181.0, 118.3)
- added G***: LOGO, locallib:ai-4.8-mask, F.Cu at (144.5, 118.3)
- added G***: LOGO, locallib:orbitx, F.Cu at (273.1, 95.2)
- moved FID3 291.0 mm to (34.1, 132.6)
- moved FID2 233.1 mm to (34.1, 19.8)
- moved J19 181.2 mm to (49.2, 112.7), turned to 180 degrees
- moved J18 169.3 mm to (276.2, 112.7), turned to 180 degrees
- moved J9 159.3 mm to (228.6, 105.6), turned to 180 degrees
- moved J5 155.0 mm to (96.8, 112.7), turned to 180 degrees
- moved J6 153.2 mm to (228.6, 112.7), turned to 180 degrees
- moved J14 148.9 mm to (96.8, 105.6), turned to 180 degrees
- moved J17 111.7 mm to (77.8, 34.9)
- moved J3 91.3 mm to (247.7, 34.9)
- moved J7 74.8 mm to (209.6, 34.9)
- moved J13 73.6 mm to (115.9, 34.9)
- moved FID1 66.0 mm to (291.3, 19.8)
- moved C1 0.52 mm to (112.9, 84.6)
- moved C2 0.52 mm to (109.1, 84.6)
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Connections:
- net LEDIND-1-R renamed Net-(U3-Pad37)
- net LEDPWM renamed Net-(U1-Pad12)
- net LEDPWM-R renamed Net-(U3-Pad12)
- net ROW4 renamed Net-(U1-Pad21)
- U1 pad 25: COL4 -> Net-(U1-Pad25)
- U1 pad 26: COL3 -> Net-(U1-Pad26)
- U1 pad 27: COL2 -> Net-(U1-Pad27)
- U1 pad 28: COL1 -> ROW0
- U1 pad 29: LEDIND-1 -> ROW1
- U1 pad 30: LEDIND-2 -> ROW2
- U1 pad 31: LEDIND-3 -> COL5
- U1 pad 32: COL0 -> COL4
- U1 pad 36: ROW0 -> ROW3
- U1 pad 37: ROW1 -> Net-(U1-Pad37)
- U1 pad 38: ROW2 -> COL3
- U1 pad 39: ROW3 -> COL2
- U1 pad 40: COL5 -> COL1
- U1 pad 41: COL6 -> COL0
- U3 pad 1: ROW4-R -> COL2-R
- U3 pad 25: COL0-R -> ROW3-R
- U3 pad 26: COL1-R -> ROW1-R
- U3 pad 27: ROW3-R -> ROW0-R
- U3 pad 28: ROW2-R -> Net-(U3-Pad28)
- U3 pad 29: ROW1-R -> Net-(U3-Pad29)
- U3 pad 30: ROW0-R -> Net-(U3-Pad30)
- U3 pad 31: COL6-R -> COL0-R
- U3 pad 32: LEDIND-3-R -> COL1-R
- U3 pad 36: LEDIND-2-R -> ROW2-R
- U3 pad 38: COL5-R -> Net-(U3-Pad38)
- U3 pad 39: COL4-R -> COL5-R
- U3 pad 40: COL2-R -> COL4-R
Routing:
- net GNDA: track 98.9 -> 281.7 mm, vias 0 -> 6
- net GND: track 148.3 -> 278.4 mm, vias 2 -> 6
- net ROW3-R: track 47.4 -> 172.7 mm, vias 0 -> 7
- net +5VA: track 23.9 -> 123.4 mm, vias 0 -> 6
- net +5V: track 76.0 -> 173.6 mm, vias 8 -> 11
- net COL5-R: track 57.1 -> 151.2 mm, vias 0 -> 3
- net COL0: track 57.1 -> 142.5 mm, vias 0 -> 2
- net SCL-R: track 3.91 -> 78.7 mm
- net COL4-R: track 57.1 -> 131.2 mm, vias 0 -> 3
- net COL1: track 59.0 -> 131.7 mm, vias 0 -> 2
- net SDA-R: track 1.97 -> 72.0 mm
- net ROW0: track 83.3 -> 145.1 mm, vias 4 -> 6
- net ROW0-R: track 83.3 -> 139.8 mm, vias 2 -> 4
- net RESET-R: track 2.64 -> 57.2 mm, vias 1 -> 3
- net COL3-R: track 57.1 -> 105.1 mm, vias 0 -> 1
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- added copper zone on B.Cu, net GND
- added copper zone on B.Cu, net GNDA
Other:
- board size 261.9 x 94.9 mm -> 261.9 x 117.5 mm
- net class POWER: trace_width 0.254 -> 0.381
- board text added: "PCB Rev 1.0 20190625 | kb.ai03.me"
- board text added: "PCB Rev 1.0 | 20190625"
- board text added: "by ai03"
