File: OrbitX-PCB/Orbit.sch (KiCad schematic (older format))
At the start: 294 parts, among them J1 PJ-3200B-4A, J10 Breakaway_Tabs, J11 PJ-3200B-4A, J12 AVR-ISP-6, J13 Breakaway_Tabs, J14 Breakaway_Tabs, J17 Breakaway_Tabs, J18 Breakaway_Tabs, J19 Breakaway_Tabs, J2 AVR-ISP-6, J20 Breakaway_Tabs, J3 Breakaway_Tabs, J5 Breakaway_Tabs, J6 Breakaway_Tabs, J7 Breakaway_Tabs, J9 Breakaway_Tabs, Q1 2N7002, Q2 2N7002, SW1 SW_Push, SW2 SW_Push, U1 ATmega32U4-MU, U2 PRTR5V0U2X, U3 ATmega32U4-MU, U4 PRTR5V0U2X, Y1 16MHz, Y2 16MHz

Commit message: Place switches, draw outline
Parts:
- removed D35, D70, D71, D72, D73, D74: LED_3mm, locallib:LED_D3.0mm, symbol Device:LED_Small
- removed D49, D50, D51, D52, D53, D54, D55, D56, D57, D58, D59, D60, D61, D62, D63, D64, D65, D66, D67, D68, D69: SOD-123, Diodes_SMD:D_SOD-123, symbol Device:D_Small
- removed MH1, MH2: HOLE, Mounting_Holes:MountingHole_5mm, symbol Connector_Generic:Conn_01x01
- removed MX1, MX10, MX11, MX12, MX13, MX14, MX15, MX16, MX17, MX18, MX19, MX2, MX20, MX21, MX22, MX23, MX24, MX25, MX26, MX27, MX28, MX29, MX3, MX30, MX31, MX32, MX33, MX35, MX36, MX37, MX38, MX39, MX4, MX40, MX41, MX42, MX43, MX44, MX45, MX46, MX47, MX48, MX49, MX5, MX50, MX51, MX52, MX53, MX54, MX55, MX56, MX57, MX58, MX59, MX6, MX60, MX61, MX62, MX64, MX65, MX66, MX67, MX68, MX7, MX8, MX9: MX-1U, MX_Alps_Hybrid:MX-1U, symbol MX_Alps_Hybrids:MX-1U
- removed MX34, MX63: MX-1.5U, MX_Alps_Hybrid:MXOnly-1.5U-Vertical, symbol MX_Alps_Hybrids:MX-1U
- removed MXA1, MXA2: ALPS-1.5U, MX_Alps_Hybrid:ALPS-1.5U, symbol MX_Alps_Hybrids:MX-1U
- removed MXE-1, MXE-2: MX-2U, MX_Alps_Hybrid:MX-2U, symbol MX_Alps_Hybrids:MX-1U
- removed MXE-3, MXE-4, MXE-5, MXE-6: MX-2U, MX_Alps_Hybrid:MX-2U-ReversedStabilizers, symbol MX_Alps_Hybrids:MX-1U
- removed Q1, Q2: 2N7002, TO_SOT_Packages_SMD:SOT-23, symbol Transistor_FET:2N7002
- removed R11, R12, R13, R14, R15, R16, R17, R18, R19, R2, R20, R21, R22, R23, R24, R26, R27, R28, R29, R3, R30, R31, R32, R34, R35, R36, R37, R38, R39, R4, R46, R47, R48, R49, R5, R50, R51, R52, R53, R54, R55, R56, R57, R58, R59, R6, R60, R61, R62, R63, R64, R65, R66, R68, R69, R7, R70, R71, R72, R73, R74, R75, R76, R77, R78, R79, R8, R80: 470, Resistors_SMD:R_0805, symbol Device:R_Small
- removed R33, R40, R81, R82, R89, R90, R91, R92: 1k, Resistors_SMD:R_0805, symbol Device:R_Small
- added D35: SOD123, Diode_SMD:D_SOD-123, symbol Device:D_Small
- added MX1, MX10, MX11, MX13, MX14, MX15, MX16, MX17, MX18, MX19, MX2, MX20, MX21, MX22, MX23, MX24, MX25, MX26, MX27, MX28, MX29, MX3, MX30, MX31, MX32, MX33, MX34, MX35, MX36, MX37, MX38, MX39, MX4, MX41, MX42, MX43, MX44, MX45, MX46, MX47, MX48, MX5, MX6, MX7, MX8, MX9: MX-NoLED, MX_Alps_Hybrid:MX-1U-NoLED, symbol MX_Alps_Hybrid:MX-NoLED
- added MX12, MX40: MX-NoLED, MX_Alps_Hybrid:MX-1.5U-NoLED, symbol MX_Alps_Hybrid:MX-NoLED
- C1, C10, C11, C12, C13, C14, C2, C3, C4, C5, C6, C7, C8, C9: footprint Capacitors_SMD:C_0603 -> Capacitor_SMD:C_0603_1608Metric
- D1, D10, D11, D12, D13, D14, D15, D16, D17, D18, D19, D2, D20, D21, D22, D23, D24, D25, D26, D27, D28, D29, D3, D30, D31, D32, D33, D34, D36, D37, D38, D39, D4, D40, D41, D42, D43, D44, D45, D46, D47, D48, D5, D6, D7, D8, D9: value SOD-123 -> SOD123; footprint Diodes_SMD:D_SOD-123 -> Diode_SMD:D_SOD-123
- D75, D76: footprint Diodes_SMD:D_SOD-123 -> Diode_SMD:D_SOD-123
- F1, F2: footprint Fuse_Holders_and_Fuses:Fuse_SMD1206_Reflow -> Fuse:Fuse_1206_3216Metric
- FID1, FID2, FID3, FID4, FID5, FID6: footprint Fiducials:Fiducial_1mm_Dia_2.54mm_Outer_CopperTop -> Fiducial:Fiducial_1mm_Dia_2.54mm_Outer_CopperTop
- J12, J2: footprint Molex-0548190589:Reset_Pretty-Mask -> random-keyboard-parts:Reset_Pretty-Mask
- R10, R25, R41, R42, R43, R44, R67, R83, R84, R85, R86, R87, R88, R9: footprint Resistors_SMD:R_0805 -> Resistor_SMD:R_0603_1608Metric
- U1, U3: footprint Housings_DFN_QFN:QFN-44-1EP_7x7mm_Pitch0.5mm -> Package_DFN_QFN:QFN-44-1EP_7x7mm_P0.5mm_EP5.2x5.2mm
- Y1, Y2: footprint Crystals:Crystal_SMD_3225-4pin_3.2x2.5mm -> Crystal:Crystal_SMD_3225-4Pin_3.2x2.5mm
Connections:
- net labels removed: LEDGND, LEDGND-R
- wire segments 653 -> 303
- no-connect marks 20 -> 18

Commit message: Progress
Connections:
- net GND: now also Y1.2, Y1.4
- net GNDA: now also Y2.2, Y2.4
Changed lines of the file:
@@
 Text GLabel 9100 11800 0    50   Input ~ 0
 ROW3-R
+Wire Wire Line
+	2650 1650 2625 1650
+Wire Wire Line
+	2425 1650 2400 1650
+Wire Wire Line
+	2650 9225 2625 9225
+Wire Wire Line
+	2425 9225 2400 9225
 $EndSCHEMATC

Commit message: Generate gerbers
Parts:
- removed FID4, FID5, FID6: Fiducial, Fiducial:Fiducial_1mm_Dia_2.54mm_Outer_CopperTop, symbol Mechanical:MountingHole
- removed J10, J20: Breakaway_Tabs, locallib:breakaway-mousebites, symbol Connector_Generic:Conn_01x01
Connections:
- net COL6 is gone; now on net COL0: U1.41 (PF0)
- net COL6-R is gone; now on net COL0-R: U3.31 (PC6)
- net LEDIND-1 is gone; now on net ROW1: U1.29 (PB5)
- net LEDIND-2 is gone; now on net ROW2: U1.30 (PB6)
- net LEDIND-2-R is gone; now on net ROW2-R: U3.36 (PF7)
- net LEDIND-3 is gone; now on net COL5: U1.31 (PC6)
- net LEDIND-3-R is gone; now on net COL1-R: U3.32 (PC7)
- net ROW4-R is gone; now on net COL2-R: U3.1 (PE6)
- net COL0: no longer U1.32 (PC7)
- net COL0-R: no longer U3.25 (PD4)
- net COL1: now also U1.40 (PF1); no longer U1.28 (PB4)
- net COL1-R: no longer U3.26 (PD6)
- net COL2: now also U1.39 (PF4); no longer U1.27 (PD7)
- net COL2-R: no longer U3.40 (PF1)
- net COL3: now also U1.38 (PF5); no longer U1.26 (PD6)
- net COL4: now also U1.32 (PC7); no longer U1.25 (PD4)
- net COL4-R: now also U3.40 (PF1); no longer U3.39 (PF4)
- net COL5: no longer U1.40 (PF1)
- net COL5-R: now also U3.39 (PF4); no longer U3.38 (PF5)
- net ROW0: now also U1.28 (PB4); no longer U1.36 (PF7)
- net ROW0-R: now also U3.27 (PD7); no longer U3.30 (PB6)
- net ROW1: no longer U1.37 (PF6)
- net ROW1-R: now also U3.26 (PD6); no longer U3.29 (PB5)
- net ROW2: no longer U1.38 (PF5)
- net ROW2-R: no longer U3.28 (PB4)
- net ROW3: now also U1.36 (PF7); no longer U1.39 (PF4)
- net ROW3-R: now also U3.25 (PD4); no longer U3.27 (PD7)
- net LEDIND-1-R: no longer names the net of U3.37 (PF6)
- net LEDPWM: no longer names the net of U1.12 (PB7)
- net LEDPWM-R: no longer names the net of U3.12 (PB7)
- net ROW4: no longer names the net of U1.21 (PD3)
- no-connect marks 18 -> 16
Changed lines of the file:
@@
 Wire Notes Line
 	675  675  675  7700
-Wire Notes Line
-	5650 675  5650 7700
 Text Notes 700  5350 0    50   ~ 0
 USB, ESD protection, Polyfuse
 Text Notes 6675 1750 0    50   ~ 0
 Resistors on left half only
-Text GLabel 4100 2050 2    50   Input ~ 0
-LEDPWM
 Text Notes 5675 4075 0    50   ~ 0
 Backlight Control
@@
 Text Notes 5675 5350 0    50   ~ 0
 Indicator LEDs\n
+Text GLabel 4100 3750 2    50   Input ~ 0
+COL0
+Text GLabel 4100 3850 2    50   Input ~ 0
+COL1
+Text GLabel 4100 3950 2    50   Input ~ 0
+COL2
+Text GLabel 4100 4050 2    50   Input ~ 0
+COL3
 Text GLabel 4100 2350 2    50   Input ~ 0
-COL0
-Text GLabel 4100 1750 2    50   Input ~ 0
-COL1
-Text GLabel 4100 3250 2    50   Input ~ 0
-COL2
-Text GLabel 4100 3150 2    50   Input ~ 0
-COL3
-Text GLabel 4100 2950 2    50   Input ~ 0
 COL4
-Text GLabel 4100 3850 2    50   Input ~ 0
+Text GLabel 4100 2250 2    50   Input ~ 0
 COL5
 Connection ~ 2900 1350
@@
 Wire Wire Line
 	4500 3450 4100 3450
-Text GLabel 4100 3750 2    50   Input ~ 0
-COL6
+Text GLabel 4100 1750 2    50   Input ~ 0
+ROW0
+Text GLabel 4100 1850 2    50   Input ~ 0
+ROW1
+Text GLabel 4100 1950 2    50   Input ~ 0
+ROW2
 Text GLabel 4100 4250 2    50   Input ~ 0
-ROW0
-Text GLabel 4100 4150 2    50   Input ~ 0
-ROW1
-Text GLabel 4100 4050 2    50   Input ~ 0
-ROW2
-Text GLabel 4100 3950 2    50   Input ~ 0
 ROW3
-Text GLabel 4100 2850 2    50   Input ~ 0
-ROW4
-Text GLabel 4100 1850 2    50   Input ~ 0
-LEDIND-1
 Wire Notes Line
 	7750 675  7750 7700
@@
 	1    0    0    -1
 $EndComp
-$Comp
-L Connector_Generic:Conn_01x01 J6
-U 1 1 5BBF48DE
-P 6000 7175
-F 0 "J6" H 6079 7217 50  0000 L CNN
-F 1 "Breakaway_Tabs" H 6079 7126 50  0000 L CNN
-F 2 "locallib:breakaway-mousebites" H 6000 7175 50  0001 C CNN
-F 3 "~" H 6000 7175 50  0001 C CNN
-	1    6000 7175
-	1    0    0    -1
-$EndComp
-NoConn ~ 5800 7175
 NoConn ~ 5800 7000
 $Comp
@@
 	1    0    0    -1
 $EndComp
-$Comp
-L Connector_Generic:Conn_01x01 J10
-U 1 1 5BC3C176
-P 6975 7175
-F 0 "J10" H 7054 7217 50  0000 L CNN
-F 1 "Breakaway_Tabs" H 7054 7126 50  0000 L CNN
-F 2 "locallib:breakaway-mousebites" H 6975 7175 50  0001 C CNN
-F 3 "~" H 6975 7175 50  0001 C CNN
-	1    6975 7175
-	1    0    0    -1
-$EndComp
-NoConn ~ 6775 7175
 NoConn ~ 6775 7000
 $Comp
@@
 Text Notes 5975 9375 0    50   ~ 0
 Resistors on left half only
-Text GLabel 4100 9625 2    50   Input ~ 0
-LEDPWM-R
 Text Notes 5675 11650 0    50   ~ 0
 Backlight Control
@@
 Text Notes 5675 12925 0    50   ~ 0
 Indicator LEDs\n
-Text GLabel 4100 10525 2    50   Input ~ 0
+Text GLabel 4100 9825 2    50   Input ~ 0
 COL0-R
-Text GLabel 4100 10725 2    50   Input ~ 0
+Text GLabel 4100 9925 2    50   Input ~ 0
 COL1-R
-Text GLabel 4100 11425 2    50   Input ~ 0
+Text GLabel 4100 11125 2    50   Input ~ 0
 COL2-R
 Text GLabel 4100 11325 2    50   Input ~ 0
 COL3-R
+Text GLabel 4100 11425 2    50   Input ~ 0
+COL4-R
 Text GLabel 4100 11525 2    50   Input ~ 0
-COL4-R
-Text GLabel 4100 11625 2    50   Input ~ 0
 COL5-R
 Connection ~ 2900 8925
@@
 Wire Wire Line
 	4500 11025 4100 11025
-Text GLabel 4100 9825 2    50   Input ~ 0
-COL6-R
-Text GLabel 4100 9525 2    50   Input ~ 0
+Text GLabel 4100 10825 2    50   Input ~ 0
 ROW0-R
-Text GLabel 4100 9425 2    50   Input ~ 0
+Text GLabel 4100 10725 2    50   Input ~ 0
 ROW1-R
-Text GLabel 4100 9325 2    50   Input ~ 0
+Text GLabel 4100 11825 2    50   Input ~ 0
 ROW2-R
-Text GLabel 4100 10825 2    50   Input ~ 0
+Text GLabel 4100 10525 2    50   Input ~ 0
 ROW3-R
-Text GLabel 4100 11125 2    50   Input ~ 0
-ROW4-R
-Text GLabel 4100 11725 2    50   Input ~ 0
-LEDIND-1-R
 Wire Notes Line
 	7750 8250 7750 15275
@@
 	1    0    0    -1
 $EndComp
-$Comp
-L Connector_Generic:Conn_01x01 J20
-U 1 1 5BCD1D70
-P 6975 14750
-F 0 "J20" H 7054 14792 50  0000 L CNN
-F 1 "Breakaway_Tabs" H 7054 14701 50  0000 L CNN
-F 2 "locallib:breakaway-mousebites" H 6975 14750 50  0001 C CNN
-F 3 "~" H 6975 14750 50  0001 C CNN
-	1    6975 14750
-	1    0    0    -1
-$EndComp
-NoConn ~ 6775 14750
 NoConn ~ 6775 14575
 Text Notes 13050 7650 0    50   ~ 10
@@
 Text GLabel 4100 10625 2    50   Input ~ 0
 HDETECT-R
-Text GLabel 4100 1950 2    50   Input ~ 0
-LEDIND-2
-Text GLabel 4100 2250 2    50   Input ~ 0
-LEDIND-3
-Text GLabel 4100 11825 2    50   Input ~ 0
-LEDIND-2-R
-Text GLabel 4100 9925 2    50   Input ~ 0
-LEDIND-3-R
 Wire Notes Line
 	14250 675  15625 675
@@
 F 3 "~" H 14400 1325 50  0001 C CNN
 	1    14400 1325
-	1    0    0    -1
-$EndComp
-$Comp
-L Mechanical:MountingHole FID4
-U 1 1 5BEFADCC
-P 15100 925
-F 0 "FID4" H 15200 971 50  0000 L CNN
-F 1 "Fiducial" H 15200 880 50  0000 L CNN
-F 2 "Fiducial:Fiducial_1mm_Dia_2.54mm_Outer_CopperTop" H 15100 925 50  0001 C CNN
-F 3 "~" H 15100 925 50  0001 C CNN
-	1    15100 925
-	1    0    0    -1
-$EndComp
-$Comp
-L Mechanical:MountingHole FID5
-U 1 1 5BEFADD3
-P 15100 1125
-F 0 "FID5" H 15200 1171 50  0000 L CNN
-F 1 "Fiducial" H 15200 1080 50  0000 L CNN
-F 2 "Fiducial:Fiducial_1mm_Dia_2.54mm_Outer_CopperTop" H 15100 1125 50  0001 C CNN
-F 3 "~" H 15100 1125 50  0001 C CNN
-	1    15100 1125
-	1    0    0    -1
-$EndComp
-$Comp
-L Mechanical:MountingHole FID6
-U 1 1 5BEFADDA
-P 15100 1325
-F 0 "FID6" H 15200 1371 50  0000 L CNN
-F 1 "Fiducial" H 15200 1280 50  0000 L CNN
-F 2 "Fiducial:Fiducial_1mm_Dia_2.54mm_Outer_CopperTop" H 15100 1325 50  0001 C CNN
-F 3 "~" H 15100 1325 50  0001 C CNN
-	1    15100 1325
 	1    0    0    -1
 $EndComp
@@
 Wire Wire Line
 	2425 9225 2400 9225
+Wire Notes Line
+	5650 675  5650 7700
+NoConn ~ 5800 7175
+$Comp
+L Connector_Generic:Conn_01x01 J6
+U 1 1 5BBF48DE
+P 6000 7175
+F 0 "J6" H 6079 7217 50  0000 L CNN
+F 1 "Breakaway_Tabs" H 6079 7126 50  0000 L CNN
+F 2 "locallib:breakaway-mousebites" H 6000 7175 50  0001 C CNN
+F 3 "~" H 6000 7175 50  0001 C CNN
+	1    6000 7175
+	1    0    0    -1
+$EndComp
 $EndSCHEMATC
